File: Hardware/Mainboard/power.kicad_sch (KiCad schematic)
At the start: 0 parts

Commit message: Adds more work on the mainboard schematic
Parts:
- added D2: 1N5822, Diode_THT:D_DO-201AD_P15.24mm_Horizontal, symbol Diode:1N5822
- added F2: 696107003002, compi:696107003002, symbol compi:696107003002
- added IC4: AOZ2261NQI-11, compi:aoz2261ngl-11, symbol compi:AOZ2261NQI-11
- added J16: 1844210, compi:combicon-1844210, symbol compi:1844210
- added SW3: SW_DPST, Button_Switch_THT:SW_Push_2P1T_Toggle_CK_PVA1xxH1xxxxxxV2, symbol Switch:SW_DPST
- added U5, U6: AZ1084CD-3.3TRG1, compi:AZ1084CD-3_3TRG1, symbol compi:AZ1084CD-3.3TRG1
Connections:
- new net: F2.1, J16.1
- new net: D2.2 (A), F2.2
- new net: J16.2, SW3.1
- new net: D2.1 (K), SW3.3
- new net +3V3: U6.2 (VO)
- new net +5V: U5.2 (VO), U6.3 (VI)
- new net +6V: IC4.16 (LX_3), IC4.17 (LX_4), IC4.18 (LX_5), U5.3 (VI)
- new net GND: IC4.12 (PGND_1), IC4.13 (PGND_2), IC4.14 (PGND_3), IC4.15 (PGND_4), IC4.4 (AGND), SW3.2, U5.1 (GND), U6.1 (GND)
- new net VCC: IC4.7 (IN_1), IC4.8 (IN_2), IC4.9 (IN_3), SW3.4
Other:
- note added: "5V => 3.3V Conversion"
- note added: "6V => 5V Conversion"
- note added: "PLACEHOLDER! Use fitting buck converter!"
- note added: "PLACEHOLDER! Use powerful 5V LDO here!"
