File: Hardware/Mainboard/Mainboard.kicad_pcb (KiCad board)
At the start: 4 copper layers, 185.4 x 160 mm, 129 parts, among them IC1 TUSB2046BIRHBR, IC2 TUSB2046BIRHBR, IC3 TUSB2046BIRHBR, IC4 AOZ2261NQI-11, J1 Conn_02x10_Odd_Even, J10 Conn_02x03_Counter_Clockwise, J11 Conn_02x03_Counter_Clockwise, J12 ARJM11D7-009-AB-EW2, J13 USB4105-GF-A-060, J14 Conn_02x03_Odd_Even, J15 Conn_02x03_Odd_Even, J16 1844210, J17 Conn_02x03_Counter_Clockwise, J18 Conn_02x03_Counter_Clockwise, J19 Conn_02x03_Counter_Clockwise, J2 Conn_02x10_Odd_Even, J20 Conn_02x03_Counter_Clockwise, J21 Conn_02x03_Counter_Clockwise, J22 Conn_02x03_Counter_Clockwise, J23 Conn_02x03_Counter_Clockwise, J3 Conn_02x10_Odd_Even, J4 Conn_02x10_Odd_Even, J5 Conn_02x10_Odd_Even, J6 Conn_02x10_Odd_Even, J7 Conn_02x10_Odd_Even, J8 Conn_02x08_Odd_Even, J9 Conn_02x12_Odd_Even, P1 USB-A1HSW6, P2 USB-A1HSW6, SW1 SW_Push_Dual, SW2 SW_Push_Dual, SW3 SW_DPST, U1 ENC624J600-I/PT, U2 SC0915, U3 CD74HC154M96, U4 TCA9548A, U5 AZ1084CD-3.3TRG1, U6 AZ1084CD-3.3TRG1, U7 RP2350_Stamp_XL

Commit message: More work on the motherboard
Parts:
- removed J13: USB4105-GF-A-060, compi:USB4105-GF-A-060
- removed U2: SC0915, compi:pi-pico
- added C25: 100n, Capacitor_SMD:C_0603_1608Metric_Pad1.08x0.95mm_HandSolder, B.Cu at (196.9, 104.8)
- added C26: 100n, Capacitor_SMD:C_0603_1608Metric_Pad1.08x0.95mm_HandSolder, B.Cu at (196.9, 107.3)
- added C27: 100n, Capacitor_SMD:C_0603_1608Metric_Pad1.08x0.95mm_HandSolder, B.Cu at (196.9, 109.8)
- added C28: 100n, Capacitor_SMD:C_0603_1608Metric_Pad1.08x0.95mm_HandSolder, B.Cu at (196.9, 112.3)
- added C29: 100n, Capacitor_SMD:C_0603_1608Metric_Pad1.08x0.95mm_HandSolder, B.Cu at (196.9, 114.8)
- added C30: 100n, Capacitor_SMD:C_0603_1608Metric_Pad1.08x0.95mm_HandSolder, B.Cu at (196.9, 117.3)
- added C31: 100n, Capacitor_SMD:C_0603_1608Metric_Pad1.08x0.95mm_HandSolder, B.Cu at (196.9, 119.8)
- added C32: 1n, Capacitor_SMD:C_0603_1608Metric_Pad1.08x0.95mm_HandSolder, B.Cu at (171.1, 105.0)
- added C33: 1n, Capacitor_SMD:C_0603_1608Metric_Pad1.08x0.95mm_HandSolder, B.Cu at (174.6, 104.4)
- added C34: 10uF, Capacitor_SMD:C_0603_1608Metric_Pad1.08x0.95mm_HandSolder, B.Cu at (170.2, 121.9)
- added C35: 6.8nF 10%, Capacitor_SMD:C_0603_1608Metric_Pad1.08x0.95mm_HandSolder, F.Cu at (172.7, 100.1)
- added C36: 6.8nF 10%, Capacitor_SMD:C_0603_1608Metric_Pad1.08x0.95mm_HandSolder, F.Cu at (172.7, 102.6)
- added C37: 10n, Capacitor_SMD:C_0603_1608Metric_Pad1.08x0.95mm_HandSolder, F.Cu at (179.3, 101.1)
- added C38: 10n, Capacitor_SMD:C_0603_1608Metric_Pad1.08x0.95mm_HandSolder, F.Cu at (179.1, 107.9)
- added R2: 49.9 1%, Resistor_SMD:R_0603_1608Metric_Pad0.98x0.95mm_HandSolder, F.Cu at (176.1, 100.1)
- added R3: 49.9 1%, Resistor_SMD:R_0603_1608Metric_Pad0.98x0.95mm_HandSolder, F.Cu at (176.1, 102.6)
- added R4: 49.9 1%, Resistor_SMD:R_0603_1608Metric_Pad0.98x0.95mm_HandSolder, F.Cu at (183.4, 97.8)
- added R5: 49.9 1%, Resistor_SMD:R_0603_1608Metric_Pad0.98x0.95mm_HandSolder, F.Cu at (183.4, 100.4)
- added R6: 10 1/12W 1%, Resistor_SMD:R_0603_1608Metric_Pad0.98x0.95mm_HandSolder, F.Cu at (183.4, 102.9)
- added U10: YC248-JR-0710KL, compi:YC248-JR-0710KL, F.Cu at (93.9, 58.9)
- added U11: YC248-JR-0710KL, compi:YC248-JR-0710KL, F.Cu at (81.2, 60.7)
- added U12: rp2040-zero, compi:rp2040-zero, F.Cu at (245.4, 59.4)
- added U8: MCP23S08T-E/SO, compi:MCP23S08T-E_SO, B.Cu at (106.1, 92.7)
- added U9: YC248-JR-0710KL, compi:YC248-JR-0710KL, F.Cu at (97.5, 90.6)
- IC1: moved to F.Cu
- moved C1 198.4 mm to (-34.6, 145.9)
- moved C10 198.4 mm to (-28.3, 126.3)
- moved C11 198.4 mm to (-2.90, 145.9)
- moved C12 198.4 mm to (-2.90, 143.4)
- moved C13 198.4 mm to (-9.25, 128.8)
- moved C14 198.4 mm to (-9.25, 126.3)
- moved C15 198.4 mm to (-28.3, 145.9)
- moved C16 198.4 mm to (-28.3, 143.4)
- moved C17 198.4 mm to (-9.25, 145.9)
- moved C18 198.4 mm to (-9.25, 143.4)
- moved C19 198.4 mm to (-15.6, 128.8)
- moved C2 198.4 mm to (-21.9, 128.8)
- moved C20 198.4 mm to (-15.6, 126.3)
- moved C21 198.4 mm to (-34.6, 128.8)
- moved C22 198.4 mm to (-34.6, 126.3)
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Connections:
- J1 pad 13: /SPI_{MISO} -> /SPI_{SCK}
- J1 pad 15: /SPI_{SCK} -> /SPI_{MOSI}
- J1 pad 17: /SPI_{MOSI} -> /SPI_{MISO}
- J12 pad 1: unconnected-(J12-Pad1) -> /Ethernet/ETH_{TX+}
- J12 pad 10: unconnected-(J12-Pad10) -> GND
- J12 pad 11: unconnected-(J12-Pad11) -> Net-(J12-Pad11)
- J12 pad 12: unconnected-(J12-Pad12) -> GND
- J12 pad 2: unconnected-(J12-Pad2) -> /Ethernet/ETH_{TX-}
- J12 pad 3: unconnected-(J12-Pad3) -> Net-(J12-RD+)
- J12 pad 4: unconnected-(J12-Pad4) -> Net-(J12-CT)
- J12 pad 5: unconnected-(J12-Pad5) -> Net-(J12-CR)
- J12 pad 6: unconnected-(J12-Pad6) -> Net-(J12-RD-)
- J12 pad 8: unconnected-(J12-Pad8) -> GND
- J12 pad 9: unconnected-(J12-Pad9) -> Net-(J12-Pad9)
- J2 pad 13: /SPI_{MISO} -> /SPI_{SCK}
- J2 pad 15: /SPI_{SCK} -> /SPI_{MOSI}
- J2 pad 17: /SPI_{MOSI} -> /SPI_{MISO}
- J3 pad 13: /SPI_{MISO} -> /SPI_{SCK}
- J3 pad 15: /SPI_{SCK} -> /SPI_{MOSI}
- J3 pad 17: /SPI_{MOSI} -> /SPI_{MISO}
- J4 pad 13: /SPI_{MISO} -> /SPI_{SCK}
- J4 pad 15: /SPI_{SCK} -> /SPI_{MOSI}
- J4 pad 17: /SPI_{MOSI} -> /SPI_{MISO}
- J5 pad 13: /SPI_{MISO} -> /SPI_{SCK}
- J5 pad 15: /SPI_{SCK} -> /SPI_{MOSI}
- J5 pad 17: /SPI_{MOSI} -> /SPI_{MISO}
- J6 pad 13: /SPI_{MISO} -> /SPI_{SCK}
- J6 pad 15: /SPI_{SCK} -> /SPI_{MOSI}
- J6 pad 17: /SPI_{MOSI} -> /SPI_{MISO}
- J7 pad 13: /SPI_{MISO} -> /SPI_{SCK}
- J7 pad 15: /SPI_{SCK} -> /SPI_{MOSI}
- J7 pad 17: /SPI_{MOSI} -> /SPI_{MISO}
- J9 pad 2: /SYS_{SCL} -> /SYS_{SDA}
- J9 pad 4: /SYS_{SDA} -> /SYS_{SCL}
- U1 pad 10: unconnected-(U1-A6-Pad10) -> GND
- U1 pad 11: unconnected-(U1-A7-Pad11) -> GND
- U1 pad 12: unconnected-(U1-A8-Pad12) -> GND
- U1 pad 13: unconnected-(U1-A9-Pad13) -> GND
- U1 pad 14: unconnected-(U1-LEDB-Pad14) -> /Ethernet/LED_{B}
- U1 pad 15: unconnected-(U1-LEDA-Pad15) -> /Ethernet/LED_{A}
- U1 pad 16: unconnected-(U1-RBIAS-Pad16) -> Net-(U1-RBIAS)
- U1 pad 17: unconnected-(U1-PSPCFG2-Pad17) -> GND
- U1 pad 18: unconnected-(U1-PSPCFG3-Pad18) -> +3V3
- U1 pad 19: unconnected-(U1-A10-Pad19) -> GND
- U1 pad 20: unconnected-(U1-A11-Pad20) -> GND
- U1 pad 21: unconnected-(U1-VDD_2-Pad21) -> +3V3
- U1 pad 22: unconnected-(U1-VDDPLL-Pad22) -> +3V3
- U1 pad 25: unconnected-(U1-VDDRX-Pad25) -> +3V3
- U1 pad 26: unconnected-(U1-TPIN+-Pad26) -> /Ethernet/ETH_{RX+}
- U1 pad 27: unconnected-(U1-TPIN--Pad27) -> /Ethernet/ETH_{RX-}
- U1 pad 28: unconnected-(U1-VDDTX-Pad28) -> +3V3
- U1 pad 3: unconnected-(U1-OSC1-Pad3) -> /Ethernet/OSC_{25MHz}
- U1 pad 30: unconnected-(U1-TPOUT+-Pad30) -> /Ethernet/ETH_{TX+}
- U1 pad 31: unconnected-(U1-TPOUT--Pad31) -> /Ethernet/ETH_{TX-}
- U1 pad 4: unconnected-(U1-VDDOSC-Pad4) -> +3V3
- U1 pad 42: unconnected-(U1-AD15-Pad42) -> GND
- U1 pad 43: unconnected-(U1-A12-Pad43) -> GND
- U1 pad 44: unconnected-(U1-A13-Pad44) -> GND
- U1 pad 45: unconnected-(U1-A14/PSPCFG1-Pad45) -> GND
- U1 pad 47: unconnected-(U1-VDD_3-Pad47) -> +3V3
- U1 pad 57: unconnected-(U1-A0-Pad57) -> GND
- U1 pad 58: unconnected-(U1-A1-Pad58) -> GND
- U1 pad 59: unconnected-(U1-A2-Pad59) -> GND
- U1 pad 60: unconnected-(U1-A3-Pad60) -> GND
- U1 pad 61: unconnected-(U1-A4-Pad61) -> GND
- U1 pad 63: unconnected-(U1-VCAP-Pad63) -> Net-(U1-VCAP)
- U1 pad 64: unconnected-(U1-VDD-Pad64) -> +3V3
- U1 pad 9: unconnected-(U1-A5-Pad9) -> GND
- U7 pad 30: /Ethernet/PSP_{CS} -> /Ethernet/PSP_{WR}
- U7 pad 42: /Ethernet/PSP_{WR} -> /Ethernet/PSP_{AL}
- U7 pad 58: /Ethernet/PSP_{AL} -> /Ethernet/PSP_{CS}
Routing:
- net /SPI_{MOSI}: track 0.00 -> 184.3 mm
- net /SPI_{MISO}: track 0.00 -> 180.0 mm
- net /SPI_{SCK}: track 0.00 -> 170.8 mm
- net /I2C_{SDA}: track 0.00 -> 80.5 mm, vias 0 -> 1
- net /I2C_{SCL}: track 0.00 -> 79.0 mm
- net Net-(J16-Pad2): track 0.00 -> 62.6 mm
- net /Ethernet/PSP_{WR}: track 0.00 -> 60.8 mm
- net /Ethernet/PSP_{RD}: track 0.00 -> 51.6 mm
- net /Ethernet/PSP_{CS}: track 0.00 -> 48.9 mm
- net /Ethernet/PSP_{AL}: track 0.00 -> 44.7 mm
- net /SYS_{SDA}: track 0.00 -> 41.5 mm, vias 0 -> 1
- net /Ethernet/PSP_{AD0}: track 0.00 -> 40.3 mm
- net /SYS_{SCL}: track 0.00 -> 39.2 mm, vias 0 -> 1
- net /Ethernet/PSP_{AD1}: track 0.00 -> 37.8 mm
- net /Ethernet/PSP_{AD14}: track 0.00 -> 36.4 mm
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