File: Hardware/Mainboard/debug.kicad_sch (KiCad schematic)
At the start: 4 parts, among them J13 USB4105-GF-A-060, SW1 SW_Push_Dual, SW2 SW_Push_Dual, U2 SC0915

Commit message: More work on the motherboard
Parts:
- removed J13: USB4105-GF-A-060, compi:USB4105-GF-A-060, symbol compi:USB4105-GF-A-060
- removed U2: SC0915, compi:pi-pico, symbol compi:SC0915
- added U12: rp2040-zero, compi:rp2040-zero, symbol compi:rp2040-zero
Connections:
- net +5V: now also U12.23 (5V)
- net GND: now also U12.22 (GND)
- net SWCLK: now also U12.4 (GP3)
- net SWDIO: now also U12.3 (GP2)
- net UART_{RXD}: now also U12.6 (GP5)
- net UART_{TXD}: now also U12.5 (GP4)
- no-connect marks 42 -> 17
Other:
- note removed: "Disconnect VBUS here otherwise we power the computer via the debug probe"
