File: Hardware/Mainboard/expansion.kicad_sch (KiCad schematic)
At the start: 6 parts, among them U10 YC248-JR-0710KL, U11 YC248-JR-0710KL, U3 CD74HC154M96, U4 TCA9548A, U8 MCP23S08T-E/SO, U9 YC248-JR-0710KL

Commit message: More work on the motherboard
Connections:
- net I2C6_{SCL}: now also U11.5 (R5); no longer U11.6 (R6)
- net I2C6_{SDA}: now also U11.6 (R6); no longer U11.5 (R5)
Other:
- moved on the sheet: U10, U11
Changed lines of the file:
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@@
 	(wire
 		(pts
-			(xy 59.69 59.69) (xy 73.66 59.69)
+			(xy 59.69 59.69) (xy 74.93 59.69)
 		)
 		(stroke
@@
 	(wire
 		(pts
-			(xy 91.44 52.07) (xy 96.52 52.07)
+			(xy 92.71 52.07) (xy 96.52 52.07)
 		)
 		(stroke
@@
 	(wire
 		(pts
-			(xy 62.23 77.47) (xy 73.66 77.47)
+			(xy 62.23 77.47) (xy 74.93 77.47)
 		)
 		(stroke
@@
 	(wire
 		(pts
-			(xy 91.44 77.47) (xy 96.52 77.47)
+			(xy 92.71 77.47) (xy 96.52 77.47)
 		)
 		(stroke
@@
 	(wire
 		(pts
-			(xy 91.44 41.91) (xy 96.52 41.91)
+			(xy 92.71 41.91) (xy 96.52 41.91)
 		)
 		(stroke
@@
 	(wire
 		(pts
-			(xy 91.44 67.31) (xy 96.52 67.31)
+			(xy 92.71 67.31) (xy 96.52 67.31)
 		)
 		(stroke
@@
 	(wire
 		(pts
-			(xy 59.69 44.45) (xy 73.66 44.45)
+			(xy 59.69 44.45) (xy 74.93 44.45)
 		)
 		(stroke
@@
 	(wire
 		(pts
-			(xy 59.69 52.07) (xy 73.66 52.07)
+			(xy 59.69 52.07) (xy 74.93 52.07)
 		)
 		(stroke
@@
 	(wire
 		(pts
-			(xy 91.44 74.93) (xy 96.52 74.93)
+			(xy 92.71 74.93) (xy 96.52 74.93)
 		)
 		(stroke
@@
 	(wire
 		(pts
+			(xy 59.69 67.31) (xy 74.93 67.31)
+		)
+		(stroke
+			(width 0)
+			(type default)
+		)
+	)
+	(wire
+		(pts
 			(xy 177.8 130.175) (xy 168.275 130.175)
 		)
@@
 	(wire
 		(pts
-			(xy 91.44 59.69) (xy 96.52 59.69)
+			(xy 92.71 59.69) (xy 96.52 59.69)
 		)
 		(stroke
@@
 	(wire
 		(pts
-			(xy 91.44 54.61) (xy 96.52 54.61)
+			(xy 92.71 54.61) (xy 96.52 54.61)
 		)
 		(stroke
@@
 	(wire
 		(pts
-			(xy 91.44 46.99) (xy 96.52 46.99)
+			(xy 92.71 46.99) (xy 96.52 46.99)
 		)
 		(stroke
@@
 	(wire
 		(pts
-			(xy 59.69 54.61) (xy 73.66 54.61)
+			(xy 73.66 69.85) (xy 74.93 69.85)
+		)
+		(stroke
+			(width 0)
+			(type default)
+		)
+	)
+	(wire
+		(pts
+			(xy 59.69 54.61) (xy 74.93 54.61)
 		)
 		(stroke
@@
 	(wire
 		(pts
-			(xy 59.69 41.91) (xy 73.66 41.91)
+			(xy 59.69 41.91) (xy 74.93 41.91)
 		)
 		(stroke
@@
 	(wire
 		(pts
-			(xy 91.44 72.39) (xy 96.52 72.39)
+			(xy 92.71 72.39) (xy 96.52 72.39)
 		)
 		(stroke
@@
 	(wire
 		(pts
-			(xy 91.44 39.37) (xy 96.52 39.37)
+			(xy 92.71 39.37) (xy 96.52 39.37)
 		)
 		(stroke
@@
 	(wire
 		(pts
-			(xy 59.69 57.15) (xy 73.66 57.15)
+			(xy 59.69 57.15) (xy 74.93 57.15)
 		)
 		(stroke
@@
 	(wire
 		(pts
-			(xy 59.69 69.85) (xy 73.66 69.85)
+			(xy 59.69 69.85) (xy 71.12 69.85)
 		)
 		(stroke
@@
 	(wire
 		(pts
-			(xy 59.69 46.99) (xy 73.66 46.99)
+			(xy 59.69 46.99) (xy 74.93 46.99)
 		)
 		(stroke
@@
 	(wire
 		(pts
-			(xy 59.69 64.77) (xy 73.66 64.77)
+			(xy 59.69 64.77) (xy 74.93 64.77)
 		)
 		(stroke
@@
 	(wire
 		(pts
-			(xy 91.44 64.77) (xy 96.52 64.77)
+			(xy 92.71 64.77) (xy 96.52 64.77)
 		)
 		(stroke
@@
 	(wire
 		(pts
-			(xy 59.69 62.23) (xy 73.66 62.23)
+			(xy 59.69 62.23) (xy 74.93 62.23)
 		)
 		(stroke
@@
 	(wire
 		(pts
+			(xy 59.69 72.39) (xy 71.12 72.39)
+		)
+		(stroke
+			(width 0)
+			(type default)
+		)
+	)
+	(wire
+		(pts
 			(xy 203.2 73.025) (xy 203.2 69.85)
 		)
@@
 	(wire
 		(pts
-			(xy 59.69 67.31) (xy 73.66 67.31)
-		)
-		(stroke
-			(width 0)
-			(type default)
-		)
-	)
-	(wire
-		(pts
 			(xy 87.63 106.68) (xy 77.47 106.68)
 		)
@@
 	(wire
 		(pts
-			(xy 59.69 72.39) (xy 73.66 72.39)
-		)
-		(stroke
-			(width 0)
-			(type default)
-		)
-	)
-	(wire
-		(pts
 			(xy 50.8 130.175) (xy 60.325 130.175)
 		)
@@
 	(wire
 		(pts
-			(xy 91.44 49.53) (xy 96.52 49.53)
+			(xy 92.71 49.53) (xy 96.52 49.53)
 		)
 		(stroke
@@
 	(wire
 		(pts
-			(xy 91.44 69.85) (xy 96.52 69.85)
+			(xy 73.66 72.39) (xy 71.12 69.85)
+		)
+		(stroke
+			(width 0)
+			(type default)
+		)
+	)
+	(wire
+		(pts
+			(xy 92.71 69.85) (xy 96.52 69.85)
 		)
 		(stroke
@@
 	(wire
 		(pts
+			(xy 73.66 69.85) (xy 71.12 72.39)
+		)
+		(stroke
+			(width 0)
+			(type default)
+		)
+	)
+	(wire
+		(pts
 			(xy 116.84 106.68) (xy 124.46 106.68)
 		)
@@
 	(wire
 		(pts
-			(xy 91.44 62.23) (xy 96.52 62.23)
+			(xy 92.71 62.23) (xy 96.52 62.23)
 		)
 		(stroke
@@
 	(wire
 		(pts
-			(xy 64.77 74.93) (xy 73.66 74.93)
+			(xy 64.77 74.93) (xy 74.93 74.93)
 		)
 		(stroke
@@
 	(wire
 		(pts
-			(xy 59.69 49.53) (xy 73.66 49.53)
+			(xy 59.69 49.53) (xy 74.93 49.53)
 		)
 		(stroke
@@
 	(wire
 		(pts
-			(xy 91.44 57.15) (xy 96.52 57.15)
+			(xy 92.71 57.15) (xy 96.52 57.15)
 		)
 		(stroke
@@
 	(wire
 		(pts
-			(xy 91.44 44.45) (xy 96.52 44.45)
+			(xy 92.71 44.45) (xy 96.52 44.45)
 		)
 		(stroke
@@
 	(wire
 		(pts
-			(xy 59.69 39.37) (xy 73.66 39.37)
+			(xy 59.69 39.37) (xy 74.93 39.37)
 		)
 		(stroke
@@
 	(wire
 		(pts
+			(xy 73.66 72.39) (xy 74.93 72.39)
+		)
+		(stroke
+			(width 0)
+			(type default)
+		)
+	)
+	(wire
+		(pts
 			(xy 215.9 152.4) (xy 206.375 152.4)
 		)
@@
 	(symbol
 		(lib_id "compi:YC248-JR-0710KL")
-		(at 82.55 48.26 0)
+		(at 83.82 48.26 0)
 		(unit 1)
 		(exclude_from_sim no)
@@
 		(dnp no)
 		(property "Reference" "U10"
-			(at 82.55 37.846 0)
+			(at 83.82 37.846 0)
 			(effects
 				(font
@@
 		)
 		(property "Value" "YC248-JR-0710KL"
-			(at 82.55 33.782 0)
+			(at 83.82 33.782 0)
 			(effects
 				(font
@@
 		)
 		(property "Footprint" "compi:YC248-JR-0710KL"
-			(at 81.28 25.4 0)
+			(at 82.55 25.4 0)
 			(effects
 				(font
@@
 		)
 		(property "Datasheet" "https://www.yageo.com/upload/media/product/app/datasheet/rchip/pyu-yc_tc_group_51_rohs_l.pdf"
-			(at 88.138 113.538 0)
+			(at 89.408 113.538 0)
 			(effects
 				(font
@@
 		)
 		(property "Description" "10k Ohm ±5% 62.5mW Power Per Element Isolated 8 Resistor Network/Array ±200ppm/°C 1606, Convex, Long Side Terminals"
-			(at 94.742 138.176 0)
+			(at 96.012 138.176 0)
 			(effects
 				(font
@@
 		)
 		(property "DigiKey Part No." "13-YC248-JR-0710KLCT-ND"
-			(at 119.38 533.02 0)
+			(at 120.65 533.02 0)
 			(effects
 				(font
@@
 		)
 		(property "TroniDex Component ID" "YC248-JR-0710KL"
-			(at 119.38 533.02 0)
+			(at 120.65 533.02 0)
 			(effects
 				(font
@@
 		)
 		(property "TroniDex Part No." "YC248-JR-0710KL"
-			(at 119.38 533.02 0)
+			(at 120.65 533.02 0)
 			(effects
 				(font
@@
 	(symbol
 		(lib_id "compi:YC248-JR-0710KL")
-		(at 82.55 68.58 0)
+		(at 83.82 68.58 0)
 		(unit 1)
 		(exclude_from_sim no)
@@
 		(dnp no)
 		(property "Reference" "U11"
-			(at 82.296 83.566 0)
+			(at 83.566 83.566 0)
 			(effects
 				(font
@@
 		)
 		(property "Value" "YC248-JR-0710KL"
-			(at 82.55 79.248 0)
+			(at 83.82 79.248 0)
 			(effects
 				(font
@@
 		)
 		(property "Footprint" "compi:YC248-JR-0710KL"
-			(at 81.28 45.72 0)
+			(at 82.55 45.72 0)
 			(effects
 				(font
@@
 		)
 		(property "Datasheet" "https://www.yageo.com/upload/media/product/app/datasheet/rchip/pyu-yc_tc_group_51_rohs_l.pdf"
-			(at 88.138 133.858 0)
+			(at 89.408 133.858 0)
 			(effects
 				(font
@@
 		)
 		(property "Description" "10k Ohm ±5% 62.5mW Power Per Element Isolated 8 Resistor Network/Array ±200ppm/°C 1606, Convex, Long Side Terminals"
-			(at 94.742 158.496 0)
+			(at 96.012 158.496 0)
 			(effects
 				(font
@@
 		)
 		(property "DigiKey Part No." "13-YC248-JR-0710KLCT-ND"
-			(at 119.38 553.34 0)
+			(at 120.65 553.34 0)
 			(effects
 				(font
@@
 		)
 		(property "TroniDex Component ID" "YC248-JR-0710KL"
-			(at 119.38 553.34 0)
+			(at 120.65 553.34 0)
 			(effects
 				(font
@@
 		)
 		(property "TroniDex Part No." "YC248-JR-0710KL"
-			(at 119.38 553.34 0)
+			(at 120.65 553.34 0)
 			(effects
 				(font
