File: Hardware/Expansions/User Expansion/PCB/Pin Cluster.kicad_sch (KiCad schematic)
At the start: 64 parts

Commit message: Continues work on User Expansion design, adds CI for exports, ERC and DRC
Parts:
- renumbered TP301 to TP601, TP202 to TP602, TP203 to TP603, TP204 to TP604, TP205 to TP605, TP206 to TP606, TP207 to TP607, TP208 to TP608, TP209 to TP609, TP210 to TP610, TP211 to TP611, TP212 to TP612, TP213 to TP613, TP214 to TP614, TP215 to TP615, TP216 to TP616, TP217 to TP617, TP218 to TP618, TP219 to TP619, TP220 to TP620, TP221 to TP621, TP222 to TP622, TP223 to TP623, TP224 to TP624, TP225 to TP625, TP226 to TP626, TP227 to TP627, TP228 to TP628, TP229 to TP629, TP230 to TP630, TP231 to TP631, TP232 to TP632, TP233 to TP633, TP234 to TP634, TP235 to TP635, TP236 to TP636, TP237 to TP637, TP238 to TP638, TP239 to TP639, TP240 to TP640, TP241 to TP641, TP242 to TP642, TP243 to TP643, TP244 to TP644, TP245 to TP645, TP246 to TP646, TP247 to TP647, TP248 to TP648, TP249 to TP649, TP250 to TP650, TP251 to TP651, TP252 to TP652, TP253 to TP653, TP254 to TP654, TP255 to TP655, TP256 to TP656, TP257 to TP657, TP258 to TP658, TP259 to TP659, TP260 to TP660, TP261 to TP661, TP262 to TP662, TP263 to TP663, TP264 to TP664
Other:
- company: (none) -> Ashet Technologies
- title: (none) -> User Expansion
