File: Hardware/Expansions/User Expansion/PCB/Pin Cluster.kicad_sch (KiCad schematic)
At the start: 64 parts

Commit message: Overhauls user expansion and updates design to new platform decisions.
Parts:
- renumbered TP601 to TP201, TP602 to TP202, TP603 to TP203, TP604 to TP204, TP605 to TP205, TP606 to TP206, TP607 to TP207, TP608 to TP208, TP609 to TP209, TP610 to TP210, TP611 to TP211, TP612 to TP212, TP613 to TP213, TP614 to TP214, TP615 to TP215, TP616 to TP216, TP617 to TP217, TP618 to TP218, TP619 to TP219, TP620 to TP220, TP621 to TP221, TP622 to TP222, TP623 to TP223, TP624 to TP224, TP625 to TP225, TP626 to TP226, TP627 to TP227, TP628 to TP228, TP629 to TP229, TP630 to TP230, TP631 to TP231, TP632 to TP232, TP633 to TP233, TP634 to TP234, TP635 to TP235, TP636 to TP236, TP637 to TP237, TP638 to TP238, TP639 to TP239, TP640 to TP240, TP641 to TP241, TP642 to TP242, TP643 to TP243, TP644 to TP244, TP645 to TP245, TP646 to TP246, TP647 to TP247, TP648 to TP248, TP649 to TP249, TP650 to TP250, TP651 to TP251, TP652 to TP252, TP653 to TP253, TP654 to TP254, TP655 to TP255, TP656 to TP256, TP657 to TP257, TP658 to TP258, TP659 to TP259, TP660 to TP260, TP661 to TP261, TP662 to TP262, TP663 to TP263, TP664 to TP264
