File: Hardware/Expansions/User Expansion/PCB/connected_row.kicad_sch (KiCad schematic)
At the start: 32 parts

Commit message: Overhauls user expansion and updates design to new platform decisions.
Parts:
- removed TP1330, TP1331, TP1332: -, TestPoint:TestPoint_THTPad_D1.5mm_Drill0.7mm, symbol Connector:TestPoint_Small
- TP1301, TP1302, TP1303, TP1304, TP1305, TP1306, TP1307, TP1308, TP1309, TP1310, TP1311, TP1312, TP1313, TP1314, TP1315, TP1316, TP1317, TP1318, TP1319, TP1320, TP1321, TP1322, TP1323, TP1324, TP1325, TP1326, TP1327, TP1328, TP1329: footprint TestPoint:TestPoint_THTPad_D1.5mm_Drill0.7mm -> Home Computer:Perfboard_Pad_P2.54mm
