File: Hardware/Backplane/Backplane.kicad_pcb (KiCad board)
At the start: 4 copper layers, 230 x 100 mm, 29 parts, among them J101 10018784-10201TLF, J201 10018784-10201TLF, J301 10018784-10201TLF, J401 10018784-10201TLF, J501 10018784-10201TLF, J601 10018784-10201TLF, J701 10018784-10201TLF, J801 10018784-10201TLF, U201 SN74LVC2G66DCUR, U202 SN74LVC2G66DCUR, U203 SN74LVC2G66DCUR, U301 SN74LVC2G66DCUR, U302 SN74LVC2G66DCUR, U303 SN74LVC2G66DCUR, U401 SN74LVC2G66DCUR, U402 SN74LVC2G66DCUR, U403 SN74LVC2G66DCUR, U501 SN74LVC2G66DCUR, U502 SN74LVC2G66DCUR, U503 SN74LVC2G66DCUR, U601 SN74LVC2G66DCUR, U602 SN74LVC2G66DCUR, U603 SN74LVC2G66DCUR, U701 SN74LVC2G66DCUR, U702 SN74LVC2G66DCUR, U703 SN74LVC2G66DCUR, U801 SN74LVC2G66DCUR, U802 SN74LVC2G66DCUR, U803 SN74LVC2G66DCUR

Commit message: Adds more work on the backplane.
Parts:
- added U101: P2X8C4M64P, Home Computer:QFP50P1600X1600X120-101N, B.Cu at (144.3, 122.2)
- U301, U302, U303, U401, U402, U403, U501, U502, U503, U601, U602, U603, U701, U702, U703, U801, U802, U803: moved to B.Cu
- moved U701 172.3 mm to (63.2, 8.30)
- moved U702 165.2 mm to (66.7, 8.30)
- moved U703 158.1 mm to (70.3, 8.30)
- moved U301 143.4 mm to (221.0, 28.0), turned to 180 degrees
- moved U302 143.4 mm to (221.0, 31.6), turned to 180 degrees
- moved U303 143.4 mm to (221.0, 35.1), turned to 180 degrees
- moved U801 126.0 mm to (86.3, 8.30)
- moved U802 118.9 mm to (89.9, 8.30)
- moved U803 111.8 mm to (93.4, 8.30)
- moved U401 88.7 mm to (193.7, 36.5)
- moved U603 84.9 mm to (106.9, 39.5)
- moved U402 81.6 mm to (190.1, 36.5)
- moved U602 77.8 mm to (110.4, 39.5)
- moved U403 74.5 mm to (186.6, 36.5)
- moved U601 70.7 mm to (114.0, 39.5)
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
Commit message: Improves Backplane Schematic a lot
Parts:
- removed J101: 10018784-10201TLF, Home Computer:CONN_10018784-10201TLF
- removed U201, U202, U203, U301, U302, U303, U401, U402, U403, U501, U502, U503, U601, U602, U603, U701, U702, U703, U801, U802, U803: SN74LVC2G66DCUR, Home Computer:SOP50P310X90-8N
- added C1001: 100n, Capacitor_SMD:C_0603_1608Metric, F.Cu at (72.5, 62.9)
- added C1002: 100n, Capacitor_SMD:C_0603_1608Metric, F.Cu at (72.5, 65.4)
- added C101: 100n, Capacitor_SMD:C_0603_1608Metric, F.Cu at (116.6, 77.6)
- added C102: 100n, Capacitor_SMD:C_0603_1608Metric, F.Cu at (119.1, 77.6)
- added C103: 100n, Capacitor_SMD:C_0603_1608Metric, F.Cu at (121.7, 77.6)
- added C902: 100n, Capacitor_SMD:C_0603_1608Metric, F.Cu at (201.1, 62.9)
- added C906: 100n, Capacitor_SMD:C_0603_1608Metric, F.Cu at (201.1, 65.5)
- added C907: 100n, Capacitor_SMD:C_0603_1608Metric, F.Cu at (201.1, 68.0)
- added C908: 100n, Capacitor_SMD:C_0603_1608Metric, F.Cu at (201.1, 70.5)
- added C909: 100n, Capacitor_SMD:C_0603_1608Metric, F.Cu at (201.1, 73.0)
- added C910: 100n, Capacitor_SMD:C_0603_1608Metric, F.Cu at (201.1, 75.5)
- added C911: 100n, Capacitor_SMD:C_0603_1608Metric, F.Cu at (201.1, 78.0)
- added C912: 100n, Capacitor_SMD:C_0603_1608Metric, F.Cu at (201.1, 80.5)
- added C913: 100n, Capacitor_SMD:C_0603_1608Metric, F.Cu at (201.1, 83.0)
- added C914: 100n, Capacitor_SMD:C_0603_1608Metric, F.Cu at (205.1, 62.9)
- added C915: 100n, Capacitor_SMD:C_0603_1608Metric, F.Cu at (205.1, 65.5)
- added C916: 100n, Capacitor_SMD:C_0603_1608Metric, F.Cu at (205.1, 68.0)
- added C917: 100n, Capacitor_SMD:C_0603_1608Metric, F.Cu at (205.1, 70.5)
- added C918: 100n, Capacitor_SMD:C_0603_1608Metric, F.Cu at (205.1, 73.0)
- added C919: 100n, Capacitor_SMD:C_0603_1608Metric, F.Cu at (205.1, 75.5)
- added C920: 100n, Capacitor_SMD:C_0603_1608Metric, F.Cu at (205.1, 78.0)
- added C921: 100n, Capacitor_SMD:C_0603_1608Metric, F.Cu at (205.1, 80.5)
- added C922: 100n, Capacitor_SMD:C_0603_1608Metric, F.Cu at (205.1, 83.0)
- added C923: 100n, Capacitor_SMD:C_0603_1608Metric, F.Cu at (209.1, 62.9)
- added C924: 100n, Capacitor_SMD:C_0603_1608Metric, F.Cu at (209.1, 65.5)
- added C925: 100n, Capacitor_SMD:C_0603_1608Metric, F.Cu at (209.1, 68.0)
- added C926: 100n, Capacitor_SMD:C_0603_1608Metric, F.Cu at (209.1, 70.5)
- added C927: 100n, Capacitor_SMD:C_0603_1608Metric, F.Cu at (209.1, 73.0)
- added C928: 100n, Capacitor_SMD:C_0603_1608Metric, F.Cu at (209.1, 75.5)
- added C929: 100n, Capacitor_SMD:C_0603_1608Metric, F.Cu at (209.1, 78.0)
- added C930: 100n, Capacitor_SMD:C_0603_1608Metric, F.Cu at (209.1, 80.5)
- added C931: 100n, Capacitor_SMD:C_0603_1608Metric, F.Cu at (209.1, 83.0)
- added C932: 100n, Capacitor_SMD:C_0603_1608Metric, F.Cu at (213.1, 62.9)
- added C933: 100n, Capacitor_SMD:C_0603_1608Metric, F.Cu at (213.1, 65.5)
- added C934: 100n, Capacitor_SMD:C_0603_1608Metric, F.Cu at (213.1, 68.0)
- added C935: 100n, Capacitor_SMD:C_0603_1608Metric, F.Cu at (213.1, 70.5)
- added C936: 100n, Capacitor_SMD:C_0603_1608Metric, F.Cu at (213.1, 73.0)
- added C937: 100n, Capacitor_SMD:C_0603_1608Metric, F.Cu at (213.1, 75.5)
- added D901: D_Small, Diode_SMD:D_1206_3216Metric, F.Cu at (36.9, 83.7)
- added D902: D_Small, Diode_SMD:D_1206_3216Metric, F.Cu at (33.4, 83.7)
- added D903: D_Small, Diode_SMD:D_1206_3216Metric, F.Cu at (40.5, 83.4)
- added F901: Polyfuse_Small, Fuse:Fuse_1206_3216Metric, F.Cu at (33.7, 72.7)
- added F902: Polyfuse_Small, Fuse:Fuse_1206_3216Metric, F.Cu at (37.0, 72.7)
- added F903: Polyfuse_Small, Fuse:Fuse_1206_3216Metric, F.Cu at (40.3, 72.7)
- added J1001: Conn_01x06, Connector_PinHeader_2.54mm:PinHeader_1x06_P2.54mm_Vertical, F.Cu at (104.2, 62.7)
- added J1002: Conn_01x06, Connector_PinHeader_2.54mm:PinHeader_1x06_P2.54mm_Vertical, F.Cu at (80.6, 62.6)
- added J1003: Conn_01x06, Connector_PinHeader_2.54mm:PinHeader_1x06_P2.54mm_Vertical, F.Cu at (88.1, 62.8)
- added J1004: Conn_01x06, Connector_PinHeader_2.54mm:PinHeader_1x06_P2.54mm_Vertical, F.Cu at (96.9, 62.8)
- added J901: Conn_01x05, Connector_Phoenix_MC:PhoenixContact_MCV_1,5_5-G-3.5_1x05_P3.50mm_Vertical, F.Cu at (33.7, 65.4)
- added R1001: 10K, Resistor_SMD:R_0603_1608Metric, F.Cu at (72.5, 67.9)
- added R1002: 4K7, Resistor_SMD:R_0603_1608Metric, F.Cu at (72.5, 70.4)
- added R1003: 4K7, Resistor_SMD:R_0603_1608Metric, F.Cu at (72.5, 72.9)
- added R201: 10, Resistor_SMD:R_0603_1608Metric, F.Cu at (169.0, 126.6)
- added R202: 10, Resistor_SMD:R_0603_1608Metric, F.Cu at (182.8, 126.6)
- added R203: 10, Resistor_SMD:R_0603_1608Metric, F.Cu at (182.8, 122.6)
- added R204: 1K, Resistor_SMD:R_0603_1608Metric, F.Cu at (169.0, 125.0)
- added R205: 1K, Resistor_SMD:R_0603_1608Metric, F.Cu at (169.0, 123.4)
- added R206: 1K, Resistor_SMD:R_0603_1608Metric, F.Cu at (169.0, 121.8)
- added R207: 1K, Resistor_SMD:R_0603_1608Metric, F.Cu at (169.0, 120.2)
- added R208: 4K7, Resistor_SMD:R_0603_1608Metric, F.Cu at (169.0, 118.6)
- added R209: 4K7, Resistor_SMD:R_0603_1608Metric, F.Cu at (169.0, 117.0)
- added R210: 1K, Resistor_SMD:R_0603_1608Metric, F.Cu at (182.8, 118.6)
- added R211: 1K, Resistor_SMD:R_0603_1608Metric, F.Cu at (182.8, 117.0)
- added R212: 1K, Resistor_SMD:R_0603_1608Metric, F.Cu at (182.8, 120.2)
- added R301: 10, Resistor_SMD:R_0603_1608Metric, F.Cu at (225.0, 126.6)
- added R302: 10, Resistor_SMD:R_0603_1608Metric, F.Cu at (238.8, 126.6)
- added R303: 10, Resistor_SMD:R_0603_1608Metric, F.Cu at (238.8, 122.6)
- added R304: 1K, Resistor_SMD:R_0603_1608Metric, F.Cu at (225.0, 125.0)
- added R305: 1K, Resistor_SMD:R_0603_1608Metric, F.Cu at (225.0, 123.4)
- added R306: 1K, Resistor_SMD:R_0603_1608Metric, F.Cu at (225.0, 121.8)
- added R307: 1K, Resistor_SMD:R_0603_1608Metric, F.Cu at (225.0, 120.2)
- added R308: 4K7, Resistor_SMD:R_0603_1608Metric, F.Cu at (225.0, 118.6)
- added R309: 4K7, Resistor_SMD:R_0603_1608Metric, F.Cu at (225.0, 117.0)
- added R310: 1K, Resistor_SMD:R_0603_1608Metric, F.Cu at (238.8, 118.6)
- added R311: 1K, Resistor_SMD:R_0603_1608Metric, F.Cu at (238.8, 117.0)
- added R312: 1K, Resistor_SMD:R_0603_1608Metric, F.Cu at (238.8, 120.2)
- added R401: 10, Resistor_SMD:R_0603_1608Metric, F.Cu at (85.0, 126.6)
- added R402: 10, Resistor_SMD:R_0603_1608Metric, F.Cu at (98.8, 126.6)
- added R403: 10, Resistor_SMD:R_0603_1608Metric, F.Cu at (98.8, 122.6)
- added R404: 1K, Resistor_SMD:R_0603_1608Metric, F.Cu at (85.0, 125.0)
- added R405: 1K, Resistor_SMD:R_0603_1608Metric, F.Cu at (85.0, 123.4)
- added R406: 1K, Resistor_SMD:R_0603_1608Metric, F.Cu at (85.0, 121.8)
- added R407: 1K, Resistor_SMD:R_0603_1608Metric, F.Cu at (85.0, 120.2)
- added R408: 4K7, Resistor_SMD:R_0603_1608Metric, F.Cu at (85.0, 118.6)
- added R409: 4K7, Resistor_SMD:R_0603_1608Metric, F.Cu at (85.0, 117.0)
- added R410: 1K, Resistor_SMD:R_0603_1608Metric, F.Cu at (98.8, 118.6)
- added R411: 1K, Resistor_SMD:R_0603_1608Metric, F.Cu at (98.8, 117.0)
- added R412: 1K, Resistor_SMD:R_0603_1608Metric, F.Cu at (98.8, 120.2)
- added R501: 10, Resistor_SMD:R_0603_1608Metric, F.Cu at (113.0, 126.6)
- added R502: 10, Resistor_SMD:R_0603_1608Metric, F.Cu at (126.8, 126.6)
- added R503: 10, Resistor_SMD:R_0603_1608Metric, F.Cu at (126.8, 122.6)
- added R504: 1K, Resistor_SMD:R_0603_1608Metric, F.Cu at (113.0, 125.0)
- added R505: 1K, Resistor_SMD:R_0603_1608Metric, F.Cu at (113.0, 123.4)
- added R506: 1K, Resistor_SMD:R_0603_1608Metric, F.Cu at (113.0, 121.8)
- added R507: 1K, Resistor_SMD:R_0603_1608Metric, F.Cu at (113.0, 120.2)
- added R508: 4K7, Resistor_SMD:R_0603_1608Metric, F.Cu at (113.0, 118.6)
- added R509: 4K7, Resistor_SMD:R_0603_1608Metric, F.Cu at (113.0, 117.0)
- added R510: 1K, Resistor_SMD:R_0603_1608Metric, F.Cu at (126.8, 118.6)
- added R511: 1K, Resistor_SMD:R_0603_1608Metric, F.Cu at (126.8, 117.0)
- added R512: 1K, Resistor_SMD:R_0603_1608Metric, F.Cu at (126.8, 120.2)
- added R601: 10, Resistor_SMD:R_0603_1608Metric, F.Cu at (197.0, 126.6)
- added R602: 10, Resistor_SMD:R_0603_1608Metric, F.Cu at (210.8, 126.6)
- added R603: 10, Resistor_SMD:R_0603_1608Metric, F.Cu at (210.8, 122.6)
- added R604: 1K, Resistor_SMD:R_0603_1608Metric, F.Cu at (197.0, 125.0)
- added R605: 1K, Resistor_SMD:R_0603_1608Metric, F.Cu at (197.0, 123.4)
- added R606: 1K, Resistor_SMD:R_0603_1608Metric, F.Cu at (197.0, 121.8)
- added R607: 1K, Resistor_SMD:R_0603_1608Metric, F.Cu at (197.0, 120.2)
- added R608: 4K7, Resistor_SMD:R_0603_1608Metric, F.Cu at (197.0, 118.6)
- added R609: 4K7, Resistor_SMD:R_0603_1608Metric, F.Cu at (197.0, 117.0)
- added R610: 1K, Resistor_SMD:R_0603_1608Metric, F.Cu at (210.8, 118.6)
- added R611: 1K, Resistor_SMD:R_0603_1608Metric, F.Cu at (210.8, 117.0)
- added R612: 1K, Resistor_SMD:R_0603_1608Metric, F.Cu at (210.8, 120.2)
- added R701: 10, Resistor_SMD:R_0603_1608Metric, F.Cu at (57.0, 126.6)
- added R702: 10, Resistor_SMD:R_0603_1608Metric, F.Cu at (70.8, 126.6)
- added R703: 10, Resistor_SMD:R_0603_1608Metric, F.Cu at (70.8, 122.6)
- added R704: 1K, Resistor_SMD:R_0603_1608Metric, F.Cu at (57.0, 125.0)
- added R705: 1K, Resistor_SMD:R_0603_1608Metric, F.Cu at (57.0, 123.4)
- added R706: 1K, Resistor_SMD:R_0603_1608Metric, F.Cu at (57.0, 121.8)
- added R707: 1K, Resistor_SMD:R_0603_1608Metric, F.Cu at (57.0, 120.2)
- added R708: 4K7, Resistor_SMD:R_0603_1608Metric, F.Cu at (57.0, 118.6)
- added R709: 4K7, Resistor_SMD:R_0603_1608Metric, F.Cu at (57.0, 117.0)
- added R710: 1K, Resistor_SMD:R_0603_1608Metric, F.Cu at (70.8, 118.6)
- added R711: 1K, Resistor_SMD:R_0603_1608Metric, F.Cu at (70.8, 117.0)
- added R712: 1K, Resistor_SMD:R_0603_1608Metric, F.Cu at (70.8, 120.2)
- added R801: 10, Resistor_SMD:R_0603_1608Metric, F.Cu at (141.0, 126.6)
- added R802: 10, Resistor_SMD:R_0603_1608Metric, F.Cu at (154.8, 126.6)
- added R803: 10, Resistor_SMD:R_0603_1608Metric, F.Cu at (154.8, 122.6)
- added R804: 1K, Resistor_SMD:R_0603_1608Metric, F.Cu at (141.0, 125.0)
- added R805: 1K, Resistor_SMD:R_0603_1608Metric, F.Cu at (141.0, 123.4)
- added R806: 1K, Resistor_SMD:R_0603_1608Metric, F.Cu at (141.0, 121.8)
- added R807: 1K, Resistor_SMD:R_0603_1608Metric, F.Cu at (141.0, 120.2)
- added R808: 4K7, Resistor_SMD:R_0603_1608Metric, F.Cu at (141.0, 118.6)
- added R809: 4K7, Resistor_SMD:R_0603_1608Metric, F.Cu at (141.0, 117.0)
- added R810: 1K, Resistor_SMD:R_0603_1608Metric, F.Cu at (154.8, 118.6)
- added R811: 1K, Resistor_SMD:R_0603_1608Metric, F.Cu at (154.8, 117.0)
- added R812: 1K, Resistor_SMD:R_0603_1608Metric, F.Cu at (154.8, 120.2)
- added R901: 1K, Resistor_SMD:R_0603_1608Metric, F.Cu at (213.1, 78.0)
- added R902: 36K 1%, Resistor_SMD:R_0603_1608Metric, F.Cu at (213.1, 80.5)
- added R903: 75K 1%, Resistor_SMD:R_0603_1608Metric, F.Cu at (213.1, 83.0)
- added TP101: TestPoint, TestPoint:TestPoint_Pad_D1.5mm, F.Cu at (117.2, 81.4)
- added TP102: TestPoint, TestPoint:TestPoint_Pad_D1.5mm, F.Cu at (120.7, 81.4)
- added TP103: TestPoint, TestPoint:TestPoint_Pad_D1.5mm, F.Cu at (124.2, 81.4)
- added TP104: TestPoint, TestPoint:TestPoint_Pad_D1.5mm, F.Cu at (127.8, 81.4)
- added TP901: +12V, TestPoint:TestPoint_Pad_D2.0mm, F.Cu at (33.7, 76.9)
- added TP902: +5V, TestPoint:TestPoint_Pad_D2.0mm, F.Cu at (37.1, 78.0)
- added TP903: +3V3, TestPoint:TestPoint_Pad_D2.0mm, F.Cu at (40.7, 77.8)
- added TP904: +1V8, TestPoint:TestPoint_Pad_D2.0mm, F.Cu at (222.7, 71.5)
- added TP905: +1V8, TestPoint:TestPoint_Pad_D2.0mm, F.Cu at (36.7, 89.8)
- added TP907: TestPoint_2Pole, Jumper:SolderJumper-2_P1.3mm_Open_Pad1.0x1.5mm, F.Cu at (224.7, 63.1)
- added U103: MCP23017_SO, Package_SO:SOIC-28W_7.5x17.9mm_P1.27mm, F.Cu at (147.0, 137.2)
- added U104: MCP23017_SO, Package_SO:SOIC-28W_7.5x17.9mm_P1.27mm, F.Cu at (122.3, 66.0)
- added U1101: SN74LVC1G08DBVR, Package_TO_SOT_SMD:SOT-23-5, F.Cu at (137.0, 60.6)
- added U1201: SN74LVC1G08DBVR, Package_TO_SOT_SMD:SOT-23-5, F.Cu at (168.3, 93.3)
- added U1301: SN74LVC1G08DBVR, Package_TO_SOT_SMD:SOT-23-5, F.Cu at (224.3, 93.3)
- added U1401: SN74LVC1G08DBVR, Package_TO_SOT_SMD:SOT-23-5, F.Cu at (84.3, 93.3)
- added U1501: SN74LVC1G08DBVR, Package_TO_SOT_SMD:SOT-23-5, F.Cu at (112.3, 93.3)
- added U1601: SN74LVC1G08DBVR, Package_TO_SOT_SMD:SOT-23-5, F.Cu at (196.3, 93.3)
- added U1701: SN74LVC1G08DBVR, Package_TO_SOT_SMD:SOT-23-5, F.Cu at (56.4, 93.3)
- added U1801: SN74LVC1G08DBVR, Package_TO_SOT_SMD:SOT-23-5, F.Cu at (140.3, 93.3)
- U101: moved to F.Cu
- moved J701 160.1 mm to (63.2, 127.6)
- moved J301 135.2 mm to (231.2, 127.6)
- moved J201 110.2 mm to (175.2, 127.6)
- moved J801 107.8 mm to (147.2, 127.6)
- moved J501 52.2 mm to (119.2, 127.6)
- moved J401 50.6 mm to (91.2, 127.6)
- moved U101 48.2 mm to (151.4, 74.6)
- moved J601 35.2 mm to (203.2, 127.6)
Connections:
- J201 pad A10: GND -> /I2C1_{SDA}
- J201 pad A11: GND -> /MOD^{1}_{~{IRQ}}
- J201 pad A13: GND -> CLOCK
- J201 pad A15: GND -> /MOD1_{GP0}
- J201 pad A16: GND -> /MOD1_{GP1}
- J201 pad A17: GND -> /MOD1_{GP2}
- J201 pad A18: /MOD1_{GP0} -> /MOD1_{GP3}
- J201 pad A19: /MOD1_{GP1} -> /MOD1_{GP4}
- J201 pad A2: /HSTX_{0} -> Net-(J201-+3V3_{RI})
- J201 pad A20: /MOD1_{GP2} -> /MOD1_{GP5}
- J201 pad A21: /MOD1_{GP3} -> /MOD1_{GP6}
- J201 pad A22: /MOD1_{GP4} -> /MOD1_{GP7}
- J201 pad A23: /MOD1_{GP5} -> unconnected-(J201-RES-PadA23)
- J201 pad A24: /MOD1_{GP6} -> unconnected-(J201-RES-PadA24)
- J201 pad A25: /MOD1_{GP7} -> unconnected-(J201-RES-PadA25)
- J201 pad A26: GND -> unconnected-(J201-RES-PadA26)
- J201 pad A27: /I2C1_{SCL} -> unconnected-(J201-RES-PadA27)
- J201 pad A28: /I2C1_{SDA} -> unconnected-(J201-RES-PadA28)
- J201 pad A29: /~{IRQ}_{1} -> unconnected-(J201-RES-PadA29)
- J201 pad A3: /HSTX_{1} -> +3V3
- J201 pad A30: CLK_{16MHz} -> unconnected-(J201-RES-PadA30)
- J201 pad A31: +3V3 -> /Module Slot 1/~{G_RESET}
- J201 pad A32: +5V -> GND
- J201 pad A4: /HSTX_{2} -> GND
- J201 pad A5: /HSTX_{3} -> Net-(J201-SLOT_{A0})
- J201 pad A6: /HSTX_{4} -> Net-(J201-SLOT_{A1})
- J201 pad A7: /HSTX_{5} -> Net-(J201-SLOT_{A2})
- J201 pad A8: /HSTX_{6} -> Net-(J201-SLOT_{A3})
- J201 pad A9: /HSTX_{7} -> /I2C1_{SCL}
- J201 pad B10: GND -> Net-(J201-~{SLOT_{AUDIO}})
- J201 pad B11: GND -> Net-(J201-~{SLOT_{VIDEO}})
- J201 pad B13: GND -> /HSTX_{0}
- J201 pad B14: GND -> /HSTX_{1}
- J201 pad B16: GND -> /HSTX_{2}
- J201 pad B17: GND -> /HSTX_{3}
- J201 pad B18: /Module Slot 1/BUS_{0} -> GND
- J201 pad B19: /Module Slot 1/BUS_{1} -> /HSTX_{4}
- J201 pad B2: GND -> Net-(J201-+12V_{RI})
- J201 pad B20: /Module Slot 1/BUS_{2} -> /HSTX_{5}
- J201 pad B21: /Module Slot 1/BUS_{3} -> GND
- J201 pad B22: /Module Slot 1/BUS_{4} -> /HSTX_{6}
- J201 pad B23: /Module Slot 1/BUS_{5} -> /HSTX_{7}
- J201 pad B24: unconnected-(J201-BUS_{6}-PadB24) -> GND
- J201 pad B3: GND -> +12V
- J201 pad B30: GND -> /Module Slot 1/I2S_{SDI}
- J201 pad B31: +3V3 -> GND
- J201 pad B32: +5V -> GND
- J201 pad B4: GND -> +12V
- J201 pad B5: GND -> +12V
- J201 pad B6: GND -> Net-(J201-+5V_{RI})
- J201 pad B7: GND -> +5V
- J201 pad B9: GND -> Net-(J201-~{PDET})
- J301 pad A10: GND -> /I2C2_{SDA}
- J301 pad A11: /I2S_{SDO} -> /MOD^{2}_{~{IRQ}}
- J301 pad A12: /I2S_{SDI} -> GND
- J301 pad A13: /I2S_{LRCLK} -> CLOCK
- J301 pad A14: /I2S_{BCLK} -> GND
- J301 pad A15: /I2S_{MCLK} -> /MOD2_{GP0}
- J301 pad A16: GND -> /MOD2_{GP1}
- J301 pad A17: GND -> /MOD2_{GP2}
- J301 pad A18: /MOD2_{GP0} -> /MOD2_{GP3}
- J301 pad A19: /MOD2_{GP1} -> /MOD2_{GP4}
- J301 pad A2: GND -> Net-(J301-+3V3_{RI})
- J301 pad A20: /MOD2_{GP2} -> /MOD2_{GP5}
- J301 pad A21: /MOD2_{GP3} -> /MOD2_{GP6}
- J301 pad A22: /MOD2_{GP4} -> /MOD2_{GP7}
- J301 pad A23: /MOD2_{GP5} -> unconnected-(J301-RES-PadA23)
- J301 pad A24: /MOD2_{GP6} -> unconnected-(J301-RES-PadA24)
- J301 pad A25: /MOD2_{GP7} -> unconnected-(J301-RES-PadA25)
- J301 pad A26: GND -> unconnected-(J301-RES-PadA26)
- J301 pad A27: /I2C2_{SCL} -> unconnected-(J301-RES-PadA27)
- J301 pad A28: /I2C2_{SDA} -> unconnected-(J301-RES-PadA28)
- J301 pad A29: /~{IRQ}_{2} -> unconnected-(J301-RES-PadA29)
- J301 pad A3: GND -> +3V3
- J301 pad A30: CLK_{16MHz} -> unconnected-(J301-RES-PadA30)
- J301 pad A31: +3V3 -> /Module Slot 2/~{G_RESET}
- J301 pad A32: +5V -> GND
- J301 pad A5: GND -> Net-(J301-SLOT_{A0})
- J301 pad A6: GND -> Net-(J301-SLOT_{A1})
- J301 pad A7: GND -> Net-(J301-SLOT_{A2})
- J301 pad A8: GND -> Net-(J301-SLOT_{A3})
- J301 pad A9: GND -> /I2C2_{SCL}
- J301 pad B10: GND -> Net-(J301-~{SLOT_{AUDIO}})
- J301 pad B11: GND -> Net-(J301-~{SLOT_{VIDEO}})
- J301 pad B18: /Module Slot 2/BUS_{0} -> GND
- J301 pad B19: /Module Slot 2/BUS_{1} -> GND
- J301 pad B2: GND -> Net-(J301-+12V_{RI})
- J301 pad B20: /Module Slot 2/BUS_{2} -> GND
- J301 pad B21: /Module Slot 2/BUS_{3} -> GND
- J301 pad B22: /Module Slot 2/BUS_{4} -> GND
- J301 pad B23: /Module Slot 2/BUS_{5} -> GND
- J301 pad B24: unconnected-(J301-BUS_{6}-PadB24) -> GND
- J301 pad B25: GND -> /I2S_{MCLK}
- J301 pad B27: GND -> /I2S_{LRCLK}
- J301 pad B28: GND -> /I2S_{BCLK}
- J301 pad B3: GND -> +12V
- J301 pad B30: GND -> /I2S_{SDI}
- J301 pad B31: +3V3 -> /I2S_{SDO}
- J301 pad B32: +5V -> GND
- J301 pad B4: GND -> +12V
- J301 pad B5: GND -> +12V
- J301 pad B6: GND -> Net-(J301-+5V_{RI})
- J301 pad B7: GND -> +5V
- J301 pad B9: GND -> Net-(J301-~{PDET})
- J401 pad A10: GND -> /I2C3_{SDA}
- J401 pad A11: GND -> /MOD^{3}_{~{IRQ}}
- J401 pad A13: GND -> CLOCK
- J401 pad A15: GND -> /MOD3_{GP0}
- J401 pad A16: GND -> /MOD3_{GP1}
- J401 pad A17: GND -> /MOD3_{GP2}
- J401 pad A18: /MOD3_{GP0} -> /MOD3_{GP3}
- J401 pad A19: /MOD3_{GP1} -> /MOD3_{GP4}
- J401 pad A2: GND -> Net-(J401-+3V3_{RI})
- J401 pad A20: /MOD3_{GP2} -> /MOD3_{GP5}
- J401 pad A21: /MOD3_{GP3} -> /MOD3_{GP6}
- J401 pad A22: /MOD3_{GP4} -> /MOD3_{GP7}
- J401 pad A23: /MOD3_{GP5} -> unconnected-(J401-RES-PadA23)
- J401 pad A24: /MOD3_{GP6} -> unconnected-(J401-RES-PadA24)
- J401 pad A25: /MOD3_{GP7} -> unconnected-(J401-RES-PadA25)
- J401 pad A26: GND -> unconnected-(J401-RES-PadA26)
- J401 pad A27: /I2C3_{SCL} -> unconnected-(J401-RES-PadA27)
- J401 pad A28: /I2C3_{SDA} -> unconnected-(J401-RES-PadA28)
- J401 pad A29: /~{IRQ}_{3} -> unconnected-(J401-RES-PadA29)
- J401 pad A3: GND -> +3V3
- J401 pad A30: CLK_{16MHz} -> unconnected-(J401-RES-PadA30)
- J401 pad A31: +3V3 -> /Module Slot 3/~{G_RESET}
- J401 pad A32: +5V -> GND
- J401 pad A5: GND -> Net-(J401-SLOT_{A0})
- J401 pad A6: GND -> Net-(J401-SLOT_{A1})
- J401 pad A7: GND -> Net-(J401-SLOT_{A2})
- J401 pad A8: GND -> Net-(J401-SLOT_{A3})
- J401 pad A9: GND -> /I2C3_{SCL}
- J401 pad B10: GND -> Net-(J401-~{SLOT_{AUDIO}})
- J401 pad B11: GND -> Net-(J401-~{SLOT_{VIDEO}})
- J401 pad B18: /Module Slot 3/BUS_{0} -> GND
- J401 pad B19: /Module Slot 3/BUS_{1} -> GND
- J401 pad B2: GND -> Net-(J401-+12V_{RI})
- J401 pad B20: /Module Slot 3/BUS_{2} -> GND
- J401 pad B21: /Module Slot 3/BUS_{3} -> GND
- J401 pad B22: /Module Slot 3/BUS_{4} -> GND
- J401 pad B23: /Module Slot 3/BUS_{5} -> GND
- J401 pad B24: unconnected-(J401-BUS_{6}-PadB24) -> GND
- J401 pad B3: GND -> +12V
- J401 pad B30: GND -> /Module Slot 3/I2S_{SDI}
- J401 pad B31: +3V3 -> GND
- J401 pad B32: +5V -> GND
- J401 pad B4: GND -> +12V
- J401 pad B5: GND -> +12V
- J401 pad B6: GND -> Net-(J401-+5V_{RI})
- J401 pad B7: GND -> +5V
- J401 pad B9: GND -> Net-(J401-~{PDET})
- J501 pad A10: GND -> /I2C4_{SDA}
- J501 pad A11: GND -> /MOD^{4}_{~{IRQ}}
- J501 pad A13: GND -> CLOCK
- J501 pad A15: GND -> /MOD4_{GP0}
- J501 pad A16: GND -> /MOD4_{GP1}
- J501 pad A17: GND -> /MOD4_{GP2}
- J501 pad A18: /MOD4_{GP0} -> /MOD4_{GP3}
- J501 pad A19: /MOD4_{GP1} -> /MOD4_{GP4}
- J501 pad A2: GND -> Net-(J501-+3V3_{RI})
- J501 pad A20: /MOD4_{GP2} -> /MOD4_{GP5}
- J501 pad A21: /MOD4_{GP3} -> /MOD4_{GP6}
- J501 pad A22: /MOD4_{GP4} -> /MOD4_{GP7}
- J501 pad A23: /MOD4_{GP5} -> unconnected-(J501-RES-PadA23)
- J501 pad A24: /MOD4_{GP6} -> unconnected-(J501-RES-PadA24)
- J501 pad A25: /MOD4_{GP7} -> unconnected-(J501-RES-PadA25)
- J501 pad A26: GND -> unconnected-(J501-RES-PadA26)
- J501 pad A27: /I2C4_{SCL} -> unconnected-(J501-RES-PadA27)
- J501 pad A28: /I2C4_{SDA} -> unconnected-(J501-RES-PadA28)
- J501 pad A29: /~{IRQ}_{4} -> unconnected-(J501-RES-PadA29)
- J501 pad A3: GND -> +3V3
- J501 pad A30: CLK_{16MHz} -> unconnected-(J501-RES-PadA30)
- J501 pad A31: +3V3 -> /Module Slot 4/~{G_RESET}
- J501 pad A32: +5V -> GND
- J501 pad A5: GND -> Net-(J501-SLOT_{A0})
- J501 pad A6: GND -> Net-(J501-SLOT_{A1})
- J501 pad A7: GND -> Net-(J501-SLOT_{A2})
- J501 pad A8: GND -> Net-(J501-SLOT_{A3})
- J501 pad A9: GND -> /I2C4_{SCL}
- J501 pad B10: GND -> Net-(J501-~{SLOT_{AUDIO}})
- J501 pad B11: GND -> Net-(J501-~{SLOT_{VIDEO}})
- J501 pad B18: /Module Slot 4/BUS_{0} -> GND
- J501 pad B19: /Module Slot 4/BUS_{1} -> GND
- J501 pad B2: GND -> Net-(J501-+12V_{RI})
- J501 pad B20: /Module Slot 4/BUS_{2} -> GND
- J501 pad B21: /Module Slot 4/BUS_{3} -> GND
- J501 pad B22: /Module Slot 4/BUS_{4} -> GND
- J501 pad B23: /Module Slot 4/BUS_{5} -> GND
- J501 pad B24: unconnected-(J501-BUS_{6}-PadB24) -> GND
- J501 pad B3: GND -> +12V
- J501 pad B30: GND -> /Module Slot 4/I2S_{SDI}
- J501 pad B31: +3V3 -> GND
- J501 pad B32: +5V -> GND
- J501 pad B4: GND -> +12V
- J501 pad B5: GND -> +12V
- J501 pad B6: GND -> Net-(J501-+5V_{RI})
- J501 pad B7: GND -> +5V
- J501 pad B9: GND -> Net-(J501-~{PDET})
- J601 pad A10: GND -> /I2C5_{SDA}
- J601 pad A11: GND -> /MOD^{5}_{~{IRQ}}
- J601 pad A13: GND -> CLOCK
- J601 pad A15: GND -> /MOD5_{GP0}
- J601 pad A16: GND -> /MOD5_{GP1}
- J601 pad A17: GND -> /MOD5_{GP2}
- J601 pad A18: /MOD5_{GP0} -> /MOD5_{GP3}
- J601 pad A19: /MOD5_{GP1} -> /MOD5_{GP4}
- J601 pad A2: GND -> Net-(J601-+3V3_{RI})
- J601 pad A20: /MOD5_{GP2} -> /MOD5_{GP5}
- J601 pad A21: /MOD5_{GP3} -> /MOD5_{GP6}
- J601 pad A22: /MOD5_{GP4} -> /MOD5_{GP7}
- J601 pad A23: /MOD5_{GP5} -> unconnected-(J601-RES-PadA23)
- J601 pad A24: /MOD5_{GP6} -> unconnected-(J601-RES-PadA24)
- J601 pad A25: /MOD5_{GP7} -> unconnected-(J601-RES-PadA25)
- J601 pad A26: GND -> unconnected-(J601-RES-PadA26)
- J601 pad A27: /I2C5_{SCL} -> unconnected-(J601-RES-PadA27)
- J601 pad A28: /I2C5_{SDA} -> unconnected-(J601-RES-PadA28)
- J601 pad A29: /~{IRQ}_{5} -> unconnected-(J601-RES-PadA29)
- J601 pad A3: GND -> +3V3
- J601 pad A30: CLK_{16MHz} -> unconnected-(J601-RES-PadA30)
- J601 pad A31: +3V3 -> /Module Slot 5/~{G_RESET}
- J601 pad A32: +5V -> GND
- J601 pad A5: GND -> Net-(J601-SLOT_{A0})
- J601 pad A6: GND -> Net-(J601-SLOT_{A1})
- J601 pad A7: GND -> Net-(J601-SLOT_{A2})
- J601 pad A8: GND -> Net-(J601-SLOT_{A3})
- J601 pad A9: GND -> /I2C5_{SCL}
- J601 pad B10: GND -> Net-(J601-~{SLOT_{AUDIO}})
- J601 pad B11: GND -> Net-(J601-~{SLOT_{VIDEO}})
- J601 pad B18: /Module Slot 5/BUS_{0} -> GND
- J601 pad B19: /Module Slot 5/BUS_{1} -> GND
- J601 pad B2: GND -> Net-(J601-+12V_{RI})
- J601 pad B20: /Module Slot 5/BUS_{2} -> GND
- J601 pad B21: /Module Slot 5/BUS_{3} -> GND
- J601 pad B22: /Module Slot 5/BUS_{4} -> GND
- J601 pad B23: /Module Slot 5/BUS_{5} -> GND
- J601 pad B24: unconnected-(J601-BUS_{6}-PadB24) -> GND
- J601 pad B3: GND -> +12V
- J601 pad B30: GND -> /Module Slot 5/I2S_{SDI}
- J601 pad B31: +3V3 -> GND
- J601 pad B32: +5V -> GND
- J601 pad B4: GND -> +12V
- J601 pad B5: GND -> +12V
- J601 pad B6: GND -> Net-(J601-+5V_{RI})
- J601 pad B7: GND -> +5V
- J601 pad B9: GND -> Net-(J601-~{PDET})
- J701 pad A10: GND -> /I2C6_{SDA}
- J701 pad A11: GND -> /MOD^{6}_{~{IRQ}}
- J701 pad A13: GND -> CLOCK
- J701 pad A15: GND -> /MOD6_{GP0}
- J701 pad A16: GND -> /MOD6_{GP1}
- J701 pad A17: GND -> /MOD6_{GP2}
- J701 pad A18: /MOD6_{GP0} -> /MOD6_{GP3}
- J701 pad A19: /MOD6_{GP1} -> /MOD6_{GP4}
- J701 pad A2: GND -> Net-(J701-+3V3_{RI})
- J701 pad A20: /MOD6_{GP2} -> /MOD6_{GP5}
- J701 pad A21: /MOD6_{GP3} -> /MOD6_{GP6}
- J701 pad A22: /MOD6_{GP4} -> /MOD6_{GP7}
- J701 pad A23: /MOD6_{GP5} -> unconnected-(J701-RES-PadA23)
- J701 pad A24: /MOD6_{GP6} -> unconnected-(J701-RES-PadA24)
- J701 pad A25: /MOD6_{GP7} -> unconnected-(J701-RES-PadA25)
- J701 pad A26: GND -> unconnected-(J701-RES-PadA26)
- J701 pad A27: /I2C6_{SCL} -> unconnected-(J701-RES-PadA27)
- J701 pad A28: /I2C6_{SDA} -> unconnected-(J701-RES-PadA28)
- J701 pad A29: /~{IRQ}_{6} -> unconnected-(J701-RES-PadA29)
- J701 pad A3: GND -> +3V3
- J701 pad A30: CLK_{16MHz} -> unconnected-(J701-RES-PadA30)
- J701 pad A31: +3V3 -> /Module Slot 6/~{G_RESET}
- J701 pad A32: +5V -> GND
- J701 pad A5: GND -> Net-(J701-SLOT_{A0})
- J701 pad A6: GND -> Net-(J701-SLOT_{A1})
- J701 pad A7: GND -> Net-(J701-SLOT_{A2})
- J701 pad A8: GND -> Net-(J701-SLOT_{A3})
- J701 pad A9: GND -> /I2C6_{SCL}
- J701 pad B10: GND -> Net-(J701-~{SLOT_{AUDIO}})
- J701 pad B11: GND -> Net-(J701-~{SLOT_{VIDEO}})
- J701 pad B18: /Module Slot 6/BUS_{0} -> GND
- J701 pad B19: /Module Slot 6/BUS_{1} -> GND
- J701 pad B2: GND -> Net-(J701-+12V_{RI})
- J701 pad B20: /Module Slot 6/BUS_{2} -> GND
- J701 pad B21: /Module Slot 6/BUS_{3} -> GND
- J701 pad B22: /Module Slot 6/BUS_{4} -> GND
- J701 pad B23: /Module Slot 6/BUS_{5} -> GND
- J701 pad B24: unconnected-(J701-BUS_{6}-PadB24) -> GND
- J701 pad B3: GND -> +12V
- J701 pad B30: GND -> /Module Slot 6/I2S_{SDI}
- J701 pad B31: +3V3 -> GND
- J701 pad B32: +5V -> GND
- J701 pad B4: GND -> +12V
- J701 pad B5: GND -> +12V
- J701 pad B6: GND -> Net-(J701-+5V_{RI})
- J701 pad B7: GND -> +5V
- J701 pad B9: GND -> Net-(J701-~{PDET})
- J801 pad A10: GND -> /I2C7_{SDA}
- J801 pad A11: GND -> /MOD^{7}_{~{IRQ}}
- J801 pad A13: GND -> CLOCK
- J801 pad A15: GND -> /MOD7_{GP0}
- J801 pad A16: GND -> /MOD7_{GP1}
- J801 pad A17: GND -> /MOD7_{GP2}
- J801 pad A18: /MOD7_{GP0} -> /MOD7_{GP3}
- J801 pad A19: /MOD7_{GP1} -> /MOD7_{GP4}
- J801 pad A2: GND -> Net-(J801-+3V3_{RI})
- J801 pad A20: /MOD7_{GP2} -> /MOD7_{GP5}
- J801 pad A21: /MOD7_{GP3} -> /MOD7_{GP6}
- J801 pad A22: /MOD7_{GP4} -> /MOD7_{GP7}
- J801 pad A23: /MOD7_{GP5} -> unconnected-(J801-RES-PadA23)
- J801 pad A24: /MOD7_{GP6} -> unconnected-(J801-RES-PadA24)
- J801 pad A25: /MOD7_{GP7} -> unconnected-(J801-RES-PadA25)
- J801 pad A26: GND -> unconnected-(J801-RES-PadA26)
- J801 pad A27: /I2C7_{SCL} -> unconnected-(J801-RES-PadA27)
- J801 pad A28: /I2C7_{SDA} -> unconnected-(J801-RES-PadA28)
- J801 pad A29: /~{IRQ}_{7} -> unconnected-(J801-RES-PadA29)
- J801 pad A3: GND -> +3V3
- J801 pad A30: CLK_{16MHz} -> unconnected-(J801-RES-PadA30)
- J801 pad A31: +3V3 -> /Module Slot 7/~{G_RESET}
- J801 pad A32: +5V -> GND
- J801 pad A5: GND -> Net-(J801-SLOT_{A0})
- J801 pad A6: GND -> Net-(J801-SLOT_{A1})
- J801 pad A7: GND -> Net-(J801-SLOT_{A2})
- J801 pad A8: GND -> Net-(J801-SLOT_{A3})
- J801 pad A9: GND -> /I2C7_{SCL}
- J801 pad B10: GND -> Net-(J801-~{SLOT_{AUDIO}})
- J801 pad B11: GND -> Net-(J801-~{SLOT_{VIDEO}})
- J801 pad B18: /Module Slot 7/BUS_{0} -> GND
- J801 pad B19: /Module Slot 7/BUS_{1} -> GND
- J801 pad B2: GND -> Net-(J801-+12V_{RI})
- J801 pad B20: /Module Slot 7/BUS_{2} -> GND
- J801 pad B21: /Module Slot 7/BUS_{3} -> GND
- J801 pad B22: /Module Slot 7/BUS_{4} -> GND
- J801 pad B23: /Module Slot 7/BUS_{5} -> GND
- J801 pad B24: unconnected-(J801-BUS_{6}-PadB24) -> GND
- J801 pad B3: GND -> +12V
- J801 pad B30: GND -> /Module Slot 7/I2S_{SDI}
- J801 pad B31: +3V3 -> GND
- J801 pad B32: +5V -> GND
- J801 pad B4: GND -> +12V
- J801 pad B5: GND -> +12V
- J801 pad B6: GND -> Net-(J801-+5V_{RI})
- J801 pad B7: GND -> +5V
- J801 pad B9: GND -> Net-(J801-~{PDET})
- U101 pad 100: ~{RESET} -> /Reset Gate/~{OUT}
- U101 pad 51: CLK_{16MHz} -> CLOCK
Routing:
- net +12V: track 0.00 -> 91.8 mm
- net +3V3: track 0.00 -> 30.3 mm, vias 0 -> 20
- net GND: track 0.14 -> 12.1 mm, vias 0 -> 8
- net /Module Slot 6/~{G_RESET}: track 0.00 -> 7.10 mm
- net /Module Slot 7/~{G_RESET}: track 0.00 -> 7.10 mm
- net /Module Slot 5/~{G_RESET}: track 0.00 -> 7.10 mm
- net /Module Slot 4/~{G_RESET}: track 0.00 -> 7.10 mm
- net /Module Slot 3/~{G_RESET}: track 0.00 -> 7.10 mm
- net /Module Slot 2/~{G_RESET}: track 0.00 -> 7.10 mm
- net /Module Slot 1/~{G_RESET}: track 0.00 -> 7.10 mm
- net Net-(J801-~{PDET}): track 0.00 -> 5.72 mm
- net Net-(J701-~{PDET}): track 0.00 -> 5.72 mm
- net Net-(J601-~{PDET}): track 0.00 -> 5.72 mm
- net Net-(J501-~{PDET}): track 0.00 -> 5.72 mm
- net Net-(J401-~{PDET}): track 0.00 -> 5.72 mm
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Other:
- board size 230 x 100 mm -> 240 x 87 mm
