File: Hardware/Backplane/Backplane.kicad_pcb (KiCad board)
At the start: 4 copper layers, 240 x 87 mm, 521 parts, among them J101 10018784-10201TLF, J1102 10018784-10201TLF, J1201 Conn_01x03, J1402 10018784-10201TLF, J1501 Conn_01x03, J1702 10018784-10201TLF, J1801 Conn_01x03, J2002 Conn_01x03, J2102 Molex 105057, J2202 Molex 105057, J2203 10018784-10201TLF, J2301 Conn_01x03, J2502 10018784-10201TLF, J2601 Conn_01x03, J2902 Conn_02x08_Counter_Clockwise, J402 10018784-10201TLF, J501 Conn_01x03, J702 10018784-10201TLF, J801 Conn_01x03, Q1004 S3134K, Q1005 S3134K, Q1101 S3134K, Q1102 GSF3407, Q1103 GSF3407, Q1104 GSF3407, Q1201 S3134K, Q1401 S3134K, Q1402 GSF3407, Q1403 GSF3407, Q1404 GSF3407, Q1501 S3134K, Q1701 S3134K, Q1702 GSF3407, Q1703 GSF3407, Q1704 GSF3407, Q1801 S3134K, Q2001 S3134K, Q2201 S3134K, Q2202 GSF3407, Q2203 GSF3407, Q2204 GSF3407, Q2301 S3134K, Q2501 S3134K, Q2502 GSF3407, Q2503 GSF3407, Q2504 GSF3407, Q2601 S3134K, Q401 S3134K, Q402 GSF3407, Q403 GSF3407, Q404 GSF3407, Q501 S3134K, Q701 S3134K, Q702 GSF3407, Q703 GSF3407, Q704 GSF3407, Q801 S3134K, SW1001 Button 12mm, U1003 CD74HC221M96, U1004 PCF8523T/1,118, U1101 NL17SZS11DFT2G-Q, U1202 CH32V003FxPx, U1203 NL17SZS11DFT2G-Q, U1401 NL17SZS11DFT2G-Q, U1502 CH32V003FxPx, U1503 NL17SZS11DFT2G-Q, U1701 NL17SZS11DFT2G-Q, U1802 CH32V003FxPx, U1803 NL17SZS11DFT2G-Q, U2001 NL17SZS11DFT2G-Q, U2004 CH32V003FxPx, U202 NL17SZS11DFT2G-Q, U203 NL17SZS11DFT2G-Q, U204 NL17SZS11DFT2G-Q, U205 NL17SZS11DFT2G-Q, U2201 NL17SZS11DFT2G-Q, U2302 CH32V003FxPx, U2303 NL17SZS11DFT2G-Q, U2501 NL17SZS11DFT2G-Q, U2602 CH32V003FxPx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

Commit message: Dumps all parts onto bcakplane layout.
Parts:
- J1501, J2102, J2202, SW1001: moved to B.Cu
- moved Q1404 367.0 mm to (247.7, 131.9), turned to 90 degrees
- moved Q1403 362.2 mm to (243.2, 131.9), turned to 90 degrees
- moved R1403 361.1 mm to (245.9, 127.4), turned to 90 degrees
- moved R1402 358.3 mm to (243.4, 127.4), turned to 90 degrees
- moved R1409 357.6 mm to (245.9, 123.4), turned to 90 degrees
- moved Q1402 357.4 mm to (238.8, 131.9), turned to 90 degrees
- moved R1401 355.6 mm to (240.9, 127.4), turned to 90 degrees
- moved R1408 354.8 mm to (243.4, 123.4), turned to 90 degrees
- moved C1405 352.9 mm to (238.4, 127.4), turned to 90 degrees
- moved Q1401 352.6 mm to (234.3, 131.9), turned to 90 degrees
- moved R1407 352.0 mm to (240.9, 123.4), turned to 90 degrees
- moved F1403 350.7 mm to (246.5, 114.6), turned to 90 degrees
- moved C1403 350.1 mm to (235.9, 127.4), turned to 90 degrees
- moved R1406 349.3 mm to (238.4, 123.4), turned to 90 degrees
- moved R1413 348.5 mm to (240.9, 119.4), turned to 90 degrees
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
Commit message: Further backplane PCB cleanup.
Parts:
- added D1006: GREEN, LED_SMD:LED_0603_1608Metric, F.Cu at (82.2, 9.11)
- added J1: 10018784-10201TLF, Home Computer:CONN_10018784-10201TLF, F.Cu at (83.7, 1.94)
- added J1003: BM04B-SRSS-TB, Connector_JST:JST_SH_BM04B-SRSS-TB_1x04-1MP_P1.00mm_Vertical, F.Cu at (80.5, 15.5)
- added J1004: BM04B-SRSS-TB, Connector_JST:JST_SH_BM04B-SRSS-TB_1x04-1MP_P1.00mm_Vertical, F.Cu at (80.5, 21.8)
- added J1005: BM04B-SRSS-TB, Connector_JST:JST_SH_BM04B-SRSS-TB_1x04-1MP_P1.00mm_Vertical, F.Cu at (80.5, 28.0)
- added J1006: BM04B-SRSS-TB, Connector_JST:JST_SH_BM04B-SRSS-TB_1x04-1MP_P1.00mm_Vertical, F.Cu at (80.5, 34.3)
- added L2901: 2.2u, Inductor_SMD:L_1008_2520Metric, F.Cu at (104.6, 25.4)
- added R1012: 560, Resistor_SMD:R_0603_1608Metric, F.Cu at (78.1, 8.60)
- added R414: 10K, Resistor_SMD:R_0603_1608Metric, F.Cu at (111.1, 33.8)
- added R415: 10K, Resistor_SMD:R_0603_1608Metric, F.Cu at (104.1, 35.1)
- added R416: 10K, Resistor_SMD:R_0603_1608Metric, F.Cu at (111.1, 24.8)
- added R417: 10K, Resistor_SMD:R_0603_1608Metric, F.Cu at (111.1, 29.3)
- added R418: 10K, Resistor_SMD:R_0603_1608Metric, F.Cu at (104.1, 30.6)
- added R419: 10K, Resistor_SMD:R_0603_1608Metric, F.Cu at (117.1, 29.3)
- added R420: 10K, Resistor_SMD:R_0603_1608Metric, F.Cu at (117.1, 24.8)
- added R421: 0, Resistor_SMD:R_0603_1608Metric, F.Cu at (78.1, -1.45)
- added R422: 0, Resistor_SMD:R_0603_1608Metric, F.Cu at (78.1, 1.06)
- added R423: 0, Resistor_SMD:R_0603_1608Metric, F.Cu at (78.1, 3.58)
- added R424: 0, Resistor_SMD:R_0603_1608Metric, F.Cu at (78.1, 6.08)
- added TP2005: TestPoint_Small, TestPoint:TestPoint_Pad_D1.0mm, F.Cu at (88.5, 25.1)
- added TP2006: TestPoint_Small, TestPoint:TestPoint_Pad_D1.0mm, F.Cu at (98.6, 25.1)
- added TP2007: TestPoint_Small, TestPoint:TestPoint_Pad_D1.0mm, F.Cu at (93.5, 25.1)
- added TP2008: TestPoint_Small, TestPoint:TestPoint_Pad_D1.0mm, F.Cu at (103.6, 13.9)
- added TP2009: TestPoint_Small, TestPoint:TestPoint_Pad_D1.0mm, F.Cu at (98.6, 13.9)
- added TP2010: TestPoint_Small, TestPoint:TestPoint_Pad_D1.0mm, F.Cu at (108.7, 13.9)
- added TP2011: TestPoint_Small, TestPoint:TestPoint_Pad_D1.0mm, F.Cu at (88.5, 13.9)
- added TP2012: TestPoint_Small, TestPoint:TestPoint_Pad_D1.0mm, F.Cu at (93.5, 13.9)
- added TP2013: TestPoint_Small, TestPoint:TestPoint_Pad_D1.0mm, F.Cu at (88.5, 28.1)
- added TP2014: TestPoint_Small, TestPoint:TestPoint_Pad_D1.0mm, F.Cu at (98.6, 28.1)
- added TP2015: TestPoint_Small, TestPoint:TestPoint_Pad_D1.0mm, F.Cu at (93.5, 28.1)
- added TP2016: TestPoint_Small, TestPoint:TestPoint_Pad_D1.0mm, F.Cu at (103.6, 17.0)
- added TP2017: TestPoint_Small, TestPoint:TestPoint_Pad_D1.0mm, F.Cu at (98.6, 17.0)
- added TP2018: TestPoint_Small, TestPoint:TestPoint_Pad_D1.0mm, F.Cu at (108.7, 17.0)
- added TP2019: TestPoint_Small, TestPoint:TestPoint_Pad_D1.0mm, F.Cu at (88.5, 17.0)
- added TP2020: TestPoint_Small, TestPoint:TestPoint_Pad_D1.0mm, F.Cu at (93.5, 17.0)
- added TP2021: TestPoint_Small, TestPoint:TestPoint_Pad_D1.0mm, F.Cu at (88.5, 31.2)
- added TP2022: TestPoint_Small, TestPoint:TestPoint_Pad_D1.0mm, F.Cu at (98.6, 31.2)
- added TP2023: TestPoint_Small, TestPoint:TestPoint_Pad_D1.0mm, F.Cu at (93.5, 31.2)
- added TP2024: TestPoint_Small, TestPoint:TestPoint_Pad_D1.0mm, F.Cu at (103.6, 20.0)
- added TP2025: TestPoint_Small, TestPoint:TestPoint_Pad_D1.0mm, F.Cu at (98.6, 20.0)
- added TP2026: TestPoint_Small, TestPoint:TestPoint_Pad_D1.0mm, F.Cu at (108.7, 20.0)
- added TP2027: TestPoint_Small, TestPoint:TestPoint_Pad_D1.0mm, F.Cu at (88.5, 20.0)
- added TP2028: TestPoint_Small, TestPoint:TestPoint_Pad_D1.0mm, F.Cu at (93.5, 20.0)
- added U201: OSC48M-3.3I/S3-20T, Crystal:Crystal_SMD_Abracon_ABM8AIG-4Pin_3.2x2.5mm, F.Cu at (114.8, 14.6)
- J1201, J1501, J1801, J2002, J2301, J2601, J501, J801: value Conn_01x03 -> BM03B-SRSS-TB; footprint Connector_Molex:Molex_PicoBlade_53047-0310_1x03_P1.25mm_Vertical -> Connector_JST:JST_SH_BM03B-SRSS-TB_1x03-1MP_P1.00mm_Vertical
- J2902: footprint Connector_PinHeader_2.54mm:PinHeader_1x16_P2.54mm_Vertical_SMD_Pin1Left -> Connector_PinHeader_2.54mm:PinHeader_2x08_P2.54mm_Vertical_SMD
- SW1001: footprint Button_Switch_THT:SW_PUSH-12mm -> Button_Switch_THT:SW_PUSH_1P1T_6x3.5mm_H4.3_APEM_MJTP1243
Connections:
- J1102 pad A8: unconnected-(J1102-RESERVED7-PadA8) -> Net-(J1102-MOD_SENSE)
- J1402 pad A8: unconnected-(J1402-RESERVED7-PadA8) -> Net-(J1402-MOD_SENSE)
- J1702 pad A8: unconnected-(J1702-RESERVED7-PadA8) -> Net-(J1702-MOD_SENSE)
- J2203 pad A8: unconnected-(J2203-RESERVED7-PadA8) -> Net-(J2203-MOD_SENSE)
- J2502 pad A8: unconnected-(J2502-RESERVED7-PadA8) -> Net-(J2502-MOD_SENSE)
- J402 pad A8: unconnected-(J402-RESERVED7-PadA8) -> Net-(J402-MOD_SENSE)
- J702 pad A8: unconnected-(J702-RESERVED7-PadA8) -> Net-(J702-MOD_SENSE)

Commit message: Backplane: Fixes missing footprints/parts, starts to work on the layout seriously.
Parts:
- removed C1101, C1103, C1105, C1401, C1403, C1405, C1701, C1703, C1705, C2201, C2203, C2205, C2501, C2503, C2505, C401, C403, C405, C701, C703, C705: 47u, Capacitor_SMD:C_0603_1608Metric
- removed J101: 10018784-10201TLF, Home Computer:CONN_10018784-10201TLF
- removed TP1104, TP1105, TP1106, TP1404, TP1405, TP1406, TP1704, TP1705, TP1706, TP2207, TP2208, TP2209, TP2504, TP2505, TP2506, TP404, TP405, TP406, TP704, TP705, TP706: TestPoint_Small, TestPoint:TestPoint_Pad_D1.0mm
- added U102: TCA9548APWR, Home Computer:TCA9548APWR, B.Cu at (47.1, 153.0)
- BT1001, C1003, C1004, C101, C1201, C1202, C1203, C1204, C1501, C1502, C1503, C1504, C1801, C1802, C1803, C1804, C2002, C201, C202, C203, C204, C205, C2301, C2302, C2303, C2304, C2601, C2602, C2603, C2604, C2901, C2902, C2903, C2904, C2905, C2906, C2907, C2908, C2909, C2910, C2911, C2912, C2913, C2914, C2915, C2916, C2917, C2918, C2919, C2920, C2921, C2922, C2923, C2924, C2925, C2926, C2927, C2928, C2929, C2930, C2931, C2932, C2933, C2934, C2935, C2936, C2937, C501, C502, C503, C504, C801, C802, C803, C804, D1001, D1003, D1004, D1005, D1006, D1101, D1401, D1701, D2201, D2501, D401, D701, F1101, F1102, F1103, F1401, F1402, F1403, F1701, F1702, F1703, F2101, F2201, F2202, F2203, F2204, F2501, F2502, F2503, F401, F402, F403, F701, F702, F703, J1003, J1004, J1005, J1006, J1201, J1801, J2002, J2301, J2601, J2902, J501, J801, L2901, NT2904, NT2905, NT2906, NT2907, Q1004, Q1005, Q1101, Q1102, Q1103, Q1104, Q1201, Q1401, Q1402, Q1403, Q1404, Q1501, Q1701, Q1702, Q1703, Q1704, Q1801, Q2001, Q2201, Q2202, Q2203, Q2204, Q2301, Q2501, Q2502, Q2503, Q2504, Q2601, Q401, Q402, Q403, Q404, Q501, Q701, Q702, Q703, Q704, Q801, R1001, R1002, R1003, R1004, R1005, R1006, R1007, R1008, R1009, R101, R1010, R1011, R1012, R1013, R1014, R1015, R1016, R102, R103, R1101, R1102, R1103, R1104, R1105, R1106, R1107, R1108, R1109, R1110, R1111, R1112, R1113, R1201, R1202, R1203, R1204, R1205, R1206, R1207, R1208, R1209, R1210, R1401, R1402, R1403, R1404, R1405, R1406, R1407, R1408, R1409, R1410, R1411, R1412, R1413, R1501, R1502, R1503, R1504, R1505, R1506, R1507, R1508, R1509, R1510, R1701, R1702, R1703, R1704, R1705, R1706, R1707, R1708, R1709, R1710, R1711, R1712, R1713, R1801, R1802, R1803, R1804, R1805, R1806, R1807, R1808, R1809, R1810, R2001, R2002, R2003, R2004, R201, R202, R203, R2102, R2103, R214, R215, R216, R217, R218, R219, R2201, R2202, R2203, R2204, R2205, R2206, R2207, R2208, R2209, R2210, R2211, R2212, R2213, R2214, R2215, R2301, R2302, R2303, R2304, R2305, R2306, R2307, R2308, R2309, R2310, R2501, R2502, R2503, R2504, R2505, R2506, R2507, R2508, R2509, R2510, R2511, R2512, R2513, R2601, R2602, R2603, R2604, R2605, R2606, R2607, R2608, R2609, R2610, R2901, R2902, R3001, R3002, R401, R402, R403, R404, R405, R406, R407, R408, R409, R410, R411, R412, R413, R414, R415, R416, R417, R418, R419, R420, R421, R422, R423, R424, R501, R502, R503, R504, R505, R506, R507, R508, R509, R510, R701, R702, R703, R704, R705, R706, R707, R708, R709, R710, R711, R712, R713, R801, R802, R803, R804, R805, R806, R807, R808, R809, R810, TP1001, TP1004, TP1005, TP1006, TP1007, TP1008, TP1009, TP1010, TP1101, TP1102, TP1103, TP1107, TP1108, TP1201, TP1202, TP1401, TP1402, TP1403, TP1407, TP1408, TP1501, TP1502, TP1701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: moved to B.Cu
- F2901, F2902, F2903: footprint Fuse:Fuse_2920_7451Metric -> Home Computer:FUSER_0ZCF0400FF2A; moved to B.Cu
- moved TP2020 213.7 mm to (248.5, 164.1), turned to 180 degrees
- moved TP2012 213.7 mm to (248.5, 161.0), turned to 180 degrees
- moved TP2028 213.7 mm to (248.5, 167.1), turned to 180 degrees
- moved SW1001 201.4 mm to (248.1, 25.1), turned to 180 degrees
- moved R3001 197.7 mm to (5.28, 119.6), turned to 180 degrees
- moved TP2019 197.6 mm to (220.5, 164.1), turned to 180 degrees
- moved TP2011 197.6 mm to (220.5, 161.0), turned to 180 degrees
- moved TP2027 197.6 mm to (220.5, 167.1), turned to 180 degrees
- moved R2510 196.5 mm to (260.2, 146.5), turned to 180 degrees
- moved Q2501 196.3 mm to (253.5, 188.8), turned to 180 degrees
- moved R2504 196.2 mm to (262.6, 114.2), turned to 0 degrees
- moved J2502 196.0 mm to (255.2, 122.5)
- moved D2501 194.5 mm to (264.2, 154.0), turned to 180 degrees
- moved R2511 194.4 mm to (260.2, 149.0), turned to 180 degrees
- moved U3001 194.1 mm to (9.26, 124.5), turned to 180 degrees
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Routing:
- net MAIN_+12V: track 0.00 -> 255.5 mm, vias 0 -> 8
- net MAIN_+5V: track 0.00 -> 238.8 mm, vias 0 -> 8
- net MAIN_+3V3: track 0.00 -> 222.5 mm, vias 0 -> 8
- net /Expansions/I2S_{SDO}: track 0.00 -> 88.8 mm
- net /Expansions/I2S_{LRCLK}: track 0.00 -> 88.7 mm
- net /Expansions/I2S_{SDI}: track 0.00 -> 88.6 mm
- net /Expansions/I2S_{BCLK}: track 0.00 -> 88.6 mm
- net /Expansions/I2S_{MCLK}: track 0.00 -> 88.5 mm
- net Net-(J2902-Pin_1): track 0.00 -> 56.0 mm, vias 0 -> 3
- net Net-(J2902-Pin_11): track 0.00 -> 52.1 mm, vias 0 -> 3
- net /Expansions/HSTX_{0}: track 0.00 -> 38.0 mm
- net /Expansions/HSTX_{4}: track 0.00 -> 38.0 mm
- net /Expansions/HSTX_{2}: track 0.00 -> 38.0 mm
- net /Expansions/HSTX_{6}: track 0.00 -> 38.0 mm
- net /Expansions/HSTX_{1}: track 0.00 -> 38.0 mm
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Other:
- board text added: "+12V"
- board text added: "+3V3"
- board text added: "+5V"
- board text added: "CPU"
- board text added: "EXP 0"
- board text added: "EXP 1"
- board text added: "EXP 2"
- board text added: "EXP 3"
- board text added: "EXP 4"
- board text added: "EXP 5"
- board text added: "EXP 6"
- board text added: "GND"
