File: Hardware/Backplane/Backplane.kicad_pcb (KiCad board)
At the start: 4 copper layers, 240 x 87 mm, 523 parts, among them J1 10018784-10201TLF, J1003 BM04B-SRSS-TB, J1004 BM04B-SRSS-TB, J1005 BM04B-SRSS-TB, J1006 BM04B-SRSS-TB, J1102 10018784-10201TLF, J1201 BM03B-SRSS-TB, J1402 10018784-10201TLF, J1501 BM03B-SRSS-TB, J1702 10018784-10201TLF, J1801 BM03B-SRSS-TB, J2002 BM03B-SRSS-TB, J2102 Molex 105057, J2202 Molex 105057, J2203 10018784-10201TLF, J2301 BM03B-SRSS-TB, J2502 10018784-10201TLF, J2601 BM03B-SRSS-TB, J2902 Conn_02x08_Counter_Clockwise, J402 10018784-10201TLF, J501 BM03B-SRSS-TB, J702 10018784-10201TLF, J801 BM03B-SRSS-TB, Q1004 S3134K, Q1005 S3134K, Q1101 S3134K, Q1102 GSF3407, Q1103 GSF3407, Q1104 GSF3407, Q1201 S3134K, Q1401 S3134K, Q1402 GSF3407, Q1403 GSF3407, Q1404 GSF3407, Q1501 S3134K, Q1701 S3134K, Q1702 GSF3407, Q1703 GSF3407, Q1704 GSF3407, Q1801 S3134K, Q2001 S3134K, Q2201 S3134K, Q2202 GSF3407, Q2203 GSF3407, Q2204 GSF3407, Q2301 S3134K, Q2501 S3134K, Q2502 GSF3407, Q2503 GSF3407, Q2504 GSF3407, Q2601 S3134K, Q401 S3134K, Q402 GSF3407, Q403 GSF3407, Q404 GSF3407, Q501 S3134K, Q701 S3134K, Q702 GSF3407, Q703 GSF3407, Q704 GSF3407, Q801 S3134K, SW1001 Button 12mm, U1003 CD74HC221M96, U1004 PCF8523T/1,118, U102 TCA9548APWR, U1101 NL17SZS11DFT2G-Q, U1202 CH32V003FxPx, U1203 NL17SZS11DFT2G-Q, U1401 NL17SZS11DFT2G-Q, U1502 CH32V003FxPx, U1503 NL17SZS11DFT2G-Q, U1701 NL17SZS11DFT2G-Q, U1802 CH32V003FxPx, U1803 NL17SZS11DFT2G-Q, U2001 NL17SZS11DFT2G-Q, U2004 CH32V003FxPx, U201 OSC48M-3.3I/S3-20T, U202 NL17SZS11DFT2G-Q, U203 NL17SZS11DFT2G-Q, U204 NL17SZS11DFT2G-Q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

Commit message: Fixes two issues regarding the power supply of the TCA9548APWR, routes TCA9548APWR.RESET to the main board controller.
Parts:
- turned U2901 to 45 degrees
Other:
- board text added: "ca. 1W bei DC ca. 2 W bei <= 1 MHz ca. 3…4 W bei 28 MHz ca. 4…6 W bei 300 MHz W=Leiterbahnbreite"
