File: Hardware/Backplane/expansions.kicad_sch (KiCad schematic)
At the start: 3 parts, among them U101 P2X8C4M64P, U102 TCA9548APWR

Commit message: Some cleanups of Backplane schematic: Adds DigiKey part numbers, removes unnecessary properties, marks test points as excluded from BOM
Parts:
- U101: Availability In Stock -> (none); Check_prices https://www.snapeda.com/parts/P2X8C4M64P/Parallax/view-part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 -> (none); Description_1 P2X8C4M64P Propeller™ Microcontroller IC 32-Bit 8-Core 180M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 -> (none); Digikey Part No (none) -> 149-P2X8C4M64P-ND; MANUFACTURER Parallax Inc. -> (none); MAXIMUM_PACKAGE_HEIGHT 1.2mm -> (none); MF Parallax Inc. -> (none); MP P2X8C4M64P -> (none); PARTREV 2022/11/01 -> (none); Package None -> (none); Price None -> (none); SNAPEDA_PN P2X8C4M64P -> (none); STANDARD IPC-7351B -> (none); SnapEDA_Link https://www.snapeda.com/parts/P2X8C4M64P/Parallax/view-part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 -> (none)
- U102: Digikey Part No (none) -> 296-34905-1-ND; MANUFACTURER Texas Instruments -> (none); MAXIMUM_PACKAGE_HEIGHT 1.2 mm -> (none); PARTREV G -> (none); STANDARD IPC-7351B -> (none)
Changed lines of the file:
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@@
 			)
 		)
-		(property "MF" "Parallax Inc."
+		(property "Digikey Part No" "149-P2X8C4M64P-ND"
 			(at 251.46 64.77 0)
 			(effects
@@
 					(size 1.27 1.27)
 				)
-				(justify bottom)
-				(hide yes)
-			)
-		)
-		(property "MAXIMUM_PACKAGE_HEIGHT" "1.2mm"
-			(at 251.46 64.77 0)
-			(effects
-				(font
-					(size 1.27 1.27)
-				)
-				(justify bottom)
-				(hide yes)
-			)
-		)
-		(property "Package" "None"
-			(at 251.46 64.77 0)
-			(effects
-				(font
-					(size 1.27 1.27)
-				)
-				(justify bottom)
-				(hide yes)
-			)
-		)
-		(property "Price" "None"
-			(at 251.46 64.77 0)
-			(effects
-				(font
-					(size 1.27 1.27)
-				)
-				(justify bottom)
-				(hide yes)
-			)
-		)
-		(property "Check_prices" "https://www.snapeda.com/parts/P2X8C4M64P/Parallax/view-part/?ref=eda"
-			(at 251.46 64.77 0)
-			(effects
-				(font
-					(size 1.27 1.27)
-				)
-				(justify bottom)
-				(hide yes)
-			)
-		)
-		(property "STANDARD" "IPC-7351B"
-			(at 251.46 64.77 0)
-			(effects
-				(font
-					(size 1.27 1.27)
-				)
-				(justify bottom)
-				(hide yes)
-			)
-		)
-		(property "PARTREV" "2022/11/01"
-			(at 251.46 64.77 0)
-			(effects
-				(font
-					(size 1.27 1.27)
-				)
-				(justify bottom)
-				(hide yes)
-			)
-		)
-		(property "SnapEDA_Link" "https://www.snapeda.com/parts/P2X8C4M64P/Parallax/view-part/?ref=snap"
-			(at 251.46 64.77 0)
-			(effects
-				(font
-					(size 1.27 1.27)
-				)
-				(justify bottom)
-				(hide yes)
-			)
-		)
-		(property "MP" "P2X8C4M64P"
-			(at 251.46 64.77 0)
-			(effects
-				(font
-					(size 1.27 1.27)
-				)
-				(justify bottom)
-				(hide yes)
-			)
-		)
-		(property "Description_1" "\n                        \n                            P2X8C4M64P Propeller™ Microcontroller IC 32-Bit 8-Core 180MHz 544KB (544K x 8) RAM 100-TQFP-EP (14x14)\n                        \n"
-			(at 251.46 64.77 0)
-			(effects
-				(font
-					(size 1.27 1.27)
-				)
-				(justify bottom)
-				(hide yes)
-			)
-		)
-		(property "SNAPEDA_PN" "P2X8C4M64P"
-			(at 251.46 64.77 0)
-			(effects
-				(font
-					(size 1.27 1.27)
-				)
-				(justify bottom)
-				(hide yes)
-			)
-		)
-		(property "Availability" "In Stock"
-			(at 251.46 64.77 0)
-			(effects
-				(font
-					(size 1.27 1.27)
-				)
-				(justify bottom)
-				(hide yes)
-			)
-		)
-		(property "MANUFACTURER" "Parallax Inc."
-			(at 251.46 64.77 0)
-			(effects
-				(font
-					(size 1.27 1.27)
-				)
-				(justify bottom)
 				(hide yes)
 			)
@@
 			)
 		)
-		(property "Datasheet" "~"
+		(property "Datasheet" ""
 			(at 202.565 125.095 0)
 			(effects
@@
 			)
 		)
-		(property "PARTREV" "G"
+		(property "Digikey Part No" "296-34905-1-ND"
 			(at 184.15 124.46 0)
 			(effects
@@
 					(size 1.27 1.27)
 				)
-				(justify bottom)
-				(hide yes)
-			)
-		)
-		(property "STANDARD" "IPC-7351B"
-			(at 184.15 124.46 0)
-			(effects
-				(font
-					(size 1.27 1.27)
-				)
-				(justify bottom)
-				(hide yes)
-			)
-		)
-		(property "MAXIMUM_PACKAGE_HEIGHT" "1.2 mm"
-			(at 184.15 124.46 0)
-			(effects
-				(font
-					(size 1.27 1.27)
-				)
-				(justify bottom)
-				(hide yes)
-			)
-		)
-		(property "MANUFACTURER" "Texas Instruments"
-			(at 184.15 124.46 0)
-			(effects
-				(font
-					(size 1.27 1.27)
-				)
-				(justify bottom)
-				(hide yes)
-			)
+				(hide yes)
+			)
