File: Hardware/Backplane/power.kicad_sch (KiCad schematic)
At the start: 57 parts, among them J2902 Conn_02x08_Counter_Clockwise, U2901 P2X8C4M64P, U2902 AP3445LW6-7

Commit message: Updates the backplane to fit the new platform definition, replaces now deprecated RTC with a new one, improves power management.
Connections:
- net MAIN_GND: now also J2902.12 (Pin_12), J2902.16 (Pin_16), J2902.4 (Pin_4), J2902.8 (Pin_8); no longer J2902.15 (Pin_15)
- net POWER_OK: now also J2902.15 (Pin_15); no longer J2902.13 (Pin_13)
- net at F2901.2, J2902.1 (Pin_1), J2902.3 (Pin_3): no longer J2902.16 (Pin_16)
- net at F2903.2, J2902.11 (Pin_11), J2902.9 (Pin_9): no longer J2902.8 (Pin_8)
- net at F2902.2, J2902.5 (Pin_5), J2902.7 (Pin_7): no longer J2902.12 (Pin_12)
