File: Hardware/Backplane/mgmt_ctrl.kicad_sch (KiCad schematic)
At the start: 23 parts, among them J501 BM03B-SRSS-TB, Q501 S3134K, U502 CH32V003FxPx, U503 NL17SZS11DFT2G-Q

Commit message: Improves backplane schematic even more
Parts:
- removed U503: NL17SZS11DFT2G-Q, Package_TO_SOT_SMD:SOT-363_SC-70-6, symbol Home Computer:NL17SZS11DFT2G-Q
- added U37: NL7SZ57DBVT1G, Package_TO_SOT_SMD:SC-74-6_1.55x2.9mm_P0.95mm, symbol Home Computer:NL7SZ57DBVT1G
Connections:
- net +3V3: now also U37.5 (VCC)
- net DAP_~{RST}: now also U37.6 (C)
- net GND: now also U37.2 (GND)
- net MGMT_~{RST}: now also U37.4 (Y)
- net ~{RESET}: now also U37.1 (B)
- net at R510.1: now also U37.3 (A)
Changed lines of the file:
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@@
 	(text_box "MGMT_~{RST} is not an open-collector signal as it's simpler to manage this way.\n\nAs we only control a single pin, that's fine."
 		(exclude_from_sim no)
-		(at 87.63 104.775 0)
+		(at 90.17 104.14 0)
 		(size 22.225 14.605)
 		(margins 0.9525 0.9525 0.9525 0.9525)
@@
 	(wire
 		(pts
-			(xy 88.9 102.87) (xy 98.425 102.87)
+			(xy 91.44 102.87) (xy 100.965 102.87)
 		)
 		(stroke
@@
 	)
 	(label "MGMT_~{RST}"
-		(at 98.425 102.87 180)
+		(at 100.965 102.87 180)
 		(effects
 			(font
@@
 	)
 	(symbol
+		(lib_id "Home Computer:NL7SZ57DBVT1G")
+		(at 83.82 102.87 0)
+		(unit 1)
+		(body_style 1)
+		(exclude_from_sim no)
+		(in_bom yes)
+		(on_board yes)
+		(in_pos_files yes)
+		(dnp no)
+		(property "Reference" "U37"
+			(at 156.21 88.8298 0)
+			(hide yes)
+			(show_name no)
+			(do_not_autoplace no)
+			(effects
+				(font
+					(size 1.27 1.27)
+				)
+			)
+		)
+		(property "Value" "NL7SZ57DBVT1G"
+			(at 156.21 91.3698 0)
+			(hide yes)
+			(show_name no)
+			(do_not_autoplace no)
+			(effects
+				(font
+					(size 1.27 1.27)
+				)
+			)
+		)
+		(property "Footprint" "Package_TO_SOT_SMD:SC-74-6_1.55x2.9mm_P0.95mm"
+			(at 89.535 125.095 0)
+			(hide yes)
+			(show_name no)
+			(do_not_autoplace no)
+			(effects
+				(font
+					(size 1.27 1.27)
+				)
+			)
+		)
+		(property "Datasheet" "https://www.onsemi.com/download/data-sheet/pdf/nl7sz57-d.pdf"
+			(at 88.9 60.325 0)
+			(hide yes)
+			(show_name no)
+			(do_not_autoplace no)
+			(effects
+				(font
+					(size 1.27 1.27)
+				)
+			)
+		)
+		(property "Description" "Configurable Multiple Function Configurable 1 Circuit 3 Input SC-74"
+			(at 88.9 60.325 0)
+			(hide yes)
+			(show_name no)
+			(do_not_autoplace no)
+			(effects
+				(font
+					(size 1.27 1.27)
+				)
+			)
+		)
+		(property "DigiKey Part No." "488-NL7SZ57DBVT1GCT-ND"
+			(at 79.375 56.515 0)
+			(hide yes)
+			(show_name no)
+			(do_not_autoplace no)
+			(effects
+				(font
+					(size 1.016 1.016)
+				)
+			)
+		)
+		(pin "3"
+		)
+		(pin "1"
+		)
+		(pin "4"
+		)
+		(pin "5"
+		)
+		(pin "2"
+		)
+		(pin "6"
+		)
+		(instances
+			(project "Backplane"
+				(path "/c6da991a-d3ed-4ac1-8b0d-12cd7ba8539b/830eb735-4083-4e97-a24b-40cca75ad59b/6ccf9da9-b2eb-4e25-a052-9a2bd1ca4ad0"
+					(reference "U42")
+					(unit 1)
+				)
+				(path "/c6da991a-d3ed-4ac1-8b0d-12cd7ba8539b/fc524bed-e1de-43ff-9b23-75610ded7ea1/0b76639d-ed2e-4d92-9374-970ebfad4ce9/8c0db8fc-3591-4cdc-ae49-7339c5352f54"
+					(reference "U40")
+					(unit 1)
+				)
+				(path "/c6da991a-d3ed-4ac1-8b0d-12cd7ba8539b/fc524bed-e1de-43ff-9b23-75610ded7ea1/34608737-04ee-4097-a679-eb9474de83e9/8c0db8fc-3591-4cdc-ae49-7339c5352f54"
+					(reference "U38")
+					(unit 1)
+				)
+				(path "/c6da991a-d3ed-4ac1-8b0d-12cd7ba8539b/fc524bed-e1de-43ff-9b23-75610ded7ea1/6a80605b-8ea1-4c9f-9925-195ca4829ff1/8c0db8fc-3591-4cdc-ae49-7339c5352f54"
+					(reference "U41")
+					(unit 1)
+				)
+				(path "/c6da991a-d3ed-4ac1-8b0d-12cd7ba8539b/fc524bed-e1de-43ff-9b23-75610ded7ea1/bd4b3b9b-7d85-45b4-9d95-7f7631822eea/8c0db8fc-3591-4cdc-ae49-7339c5352f54"
+					(reference "U39")
+					(unit 1)
+				)
+				(path "/c6da991a-d3ed-4ac1-8b0d-12cd7ba8539b/fc524bed-e1de-43ff-9b23-75610ded7ea1/c4424f84-74bb-4fe6-9366-b0d1f638ed10/8c0db8fc-3591-4cdc-ae49-7339c5352f54"
+					(reference "U44")
+					(unit 1)
+				)
+				(path "/c6da991a-d3ed-4ac1-8b0d-12cd7ba8539b/fc524bed-e1de-43ff-9b23-75610ded7ea1/d3047f77-c81c-4381-bf90-1d561e67b161/8c0db8fc-3591-4cdc-ae49-7339c5352f54"
+					(reference "U37")
+					(unit 1)
+				)
+				(path "/c6da991a-d3ed-4ac1-8b0d-12cd7ba8539b/fc524bed-e1de-43ff-9b23-75610ded7ea1/f94c2515-5da6-4862-ba30-6d4a39ae8639/8c0db8fc-3591-4cdc-ae49-7339c5352f54"
+					(reference "U43")
+					(unit 1)
+				)
+			)
+		)
+	)
+	(symbol
 		(lib_id "power:GND")
 		(at 45.72 100.33 0)
@@
 	)
 	(symbol
-		(lib_id "Home Computer:NL17SZS11DFT2G-Q")
-		(at 82.55 102.87 0)
-		(unit 1)
-		(body_style 1)
-		(exclude_from_sim no)
-		(in_bom yes)
-		(on_board yes)
-		(in_pos_files yes)
-		(dnp no)
-		(property "Reference" "U503"
-			(at 85.725 96.52 0)
-			(show_name no)
-			(do_not_autoplace no)
-			(effects
-				(font
-					(size 1.27 1.27)
-				)
-			)
-		)
-		(property "Value" "NL17SZS11DFT2G-Q"
-			(at 97.155 99.3392 0)
-			(show_name no)
-			(do_not_autoplace no)
-			(effects
-				(font
-					(size 1.27 1.27)
-				)
-			)
-		)
-		(property "Footprint" "Package_TO_SOT_SMD:SOT-363_SC-70-6"
-			(at 135.382 154.94 0)
-			(hide yes)
-			(show_name no)
-			(do_not_autoplace no)
-			(effects
-				(font
-					(size 1.27 1.27)
-				)
-			)
-		)
-		(property "Datasheet" "https://www.onsemi.com/download/data-sheet/pdf/nl17szs11-d.pdf"
-			(at 138.176 146.812 0)
-			(hide yes)
-			(show_name no)
-			(do_not_autoplace no)
-			(effects
-				(font
-					(size 1.27 1.27)
-				)
-			)
-		)
-		(property "Description" "AND Gate IC 1 Channel Schmitt Trigger Input SC-88/SC70-6/SOT-363"
-			(at 123.952 145.034 0)
-			(hide yes)
-			(show_name no)
-			(do_not_autoplace no)
-			(effects
-				(font
-					(size 1.27 1.27)
-				)
-			)
-		)
-		(property "DigiKey Part No" ""
-			(at 157.226 138.684 0)
-			(hide yes)
-			(show_name no)
-			(do_not_autoplace no)
-			(effects
-				(font
-					(size 1.016 1.016)
-				)
-			)
-		)
-		(property "Digikey Part No" "488-NL17SZS11DFT2G-QCT-ND"
-			(at 82.55 102.87 0)
-			(hide yes)
-			(show_name no)
-			(do_not_autoplace no)
-			(effects
-				(font
-					(size 1.27 1.27)
-				)
-			)
-		)
-		(pin "1"
-		)
-		(pin "3"
-		)
-		(pin "2"
-		)
-		(pin "4"
-		)
-		(pin "5"
-		)
-		(pin "6"
-		)
-		(instances
-			(project "Backplane"
-				(path "/c6da991a-d3ed-4ac1-8b0d-12cd7ba8539b/830eb735-4083-4e97-a24b-40cca75ad59b/6ccf9da9-b2eb-4e25-a052-9a2bd1ca4ad0"
-					(reference "U2001")
-					(unit 1)
-				)
-				(path "/c6da991a-d3ed-4ac1-8b0d-12cd7ba8539b/fc524bed-e1de-43ff-9b23-75610ded7ea1/0b76639d-ed2e-4d92-9374-970ebfad4ce9/8c0db8fc-3591-4cdc-ae49-7339c5352f54"
-					(reference "U1503")
-					(unit 1)
-				)
-				(path "/c6da991a-d3ed-4ac1-8b0d-12cd7ba8539b/fc524bed-e1de-43ff-9b23-75610ded7ea1/34608737-04ee-4097-a679-eb9474de83e9/8c0db8fc-3591-4cdc-ae49-7339c5352f54"
-					(reference "U803")
-					(unit 1)
-				)
-				(path "/c6da991a-d3ed-4ac1-8b0d-12cd7ba8539b/fc524bed-e1de-43ff-9b23-75610ded7ea1/6a80605b-8ea1-4c9f-9925-195ca4829ff1/8c0db8fc-3591-4cdc-ae49-7339c5352f54"
-					(reference "U1803")
-					(unit 1)
-				)
-				(path "/c6da991a-d3ed-4ac1-8b0d-12cd7ba8539b/fc524bed-e1de-43ff-9b23-75610ded7ea1/bd4b3b9b-7d85-45b4-9d95-7f7631822eea/8c0db8fc-3591-4cdc-ae49-7339c5352f54"
-					(reference "U1203")
-					(unit 1)
-				)
-				(path "/c6da991a-d3ed-4ac1-8b0d-12cd7ba8539b/fc524bed-e1de-43ff-9b23-75610ded7ea1/c4424f84-74bb-4fe6-9366-b0d1f638ed10/8c0db8fc-3591-4cdc-ae49-7339c5352f54"
-					(reference "U2603")
-					(unit 1)
-				)
-				(path "/c6da991a-d3ed-4ac1-8b0d-12cd7ba8539b/fc524bed-e1de-43ff-9b23-75610ded7ea1/d3047f77-c81c-4381-bf90-1d561e67b161/8c0db8fc-3591-4cdc-ae49-7339c5352f54"
-					(reference "U503")
-					(unit 1)
-				)
-				(path "/c6da991a-d3ed-4ac1-8b0d-12cd7ba8539b/fc524bed-e1de-43ff-9b23-75610ded7ea1/f94c2515-5da6-4862-ba30-6d4a39ae8639/8c0db8fc-3591-4cdc-ae49-7339c5352f54"
-					(reference "U2303")
-					(unit 1)
-				)
-			)
-		)
-	)
-	(symbol
 		(lib_id "power:GND")
 		(at 228.6 57.15 0)
@@
 	(symbol
 		(lib_id "power:+3V3")
-		(at 82.55 95.25 0)
+		(at 83.82 95.25 0)
 		(mirror y)
 		(unit 1)
@@
 		(dnp no)
 		(property "Reference" "#PWR0503"
-			(at 82.55 99.06 0)
+			(at 83.82 99.06 0)
 			(hide yes)
 			(show_name no)
@@
 		)
 		(property "Value" "+3V3"
-			(at 82.55 92.075 90)
+			(at 83.82 92.075 90)
 			(show_name no)
 			(do_not_autoplace no)
@@
 		)
 		(property "Footprint" ""
-			(at 82.55 95.25 0)
+			(at 83.82 95.25 0)
 			(hide yes)
 			(show_name no)
@@
 		)
 		(property "Datasheet" ""
-			(at 82.55 95.25 0)
+			(at 83.82 95.25 0)
 			(hide yes)
 			(show_name no)
@@
 		)
 		(property "Description" "Power symbol creates a global label with name \"+3V3\""
-			(at 82.55 95.25 0)
+			(at 83.82 95.25 0)
 			(hide yes)
 			(show_name no)
@@
 	(symbol
 		(lib_id "power:GND")
-		(at 82.55 110.49 0)
+		(at 83.82 110.49 0)
 		(unit 1)
 		(body_style 1)
@@
 		(fields_autoplaced yes)
 		(property "Reference" "#PWR0504"
-			(at 82.55 116.84 0)
+			(at 83.82 116.84 0)
 			(hide yes)
 			(show_name no)
@@
 		)
 		(property "Value" "GND"
-			(at 82.55 115.57 0)
+			(at 83.82 115.57 0)
 			(show_name no)
 			(do_not_autoplace no)
@@
 		)
 		(property "Footprint" ""
-			(at 82.55 110.49 0)
+			(at 83.82 110.49 0)
 			(hide yes)
 			(show_name no)
@@
 		)
 		(property "Datasheet" ""
-			(at 82.55 110.49 0)
+			(at 83.82 110.49 0)
 			(hide yes)
 			(show_name no)
@@
 		)
 		(property "Description" "Power symbol creates a global label with name \"GND\" , ground"
-			(at 82.55 110.49 0)
+			(at 83.82 110.49 0)
 			(hide yes)
 			(show_name no)

Commit message: Starts to work on the first Backplane sub-schematic prototype
Parts:
- renumbered C501 to C6, C502 to C7, C503 to C8, C504 to C9, J501 to J2, Q501 to Q3, R509 to R19, R508 to R20, R501 to R21, R510 to R22, R502 to R23, R503 to R24, R504 to R25, R505 to R26, R506 to R27, R507 to R28, TP2013 to TP10, TP2021 to TP11, TP501 to TP7, TP502 to TP8, TP2005 to TP9, U37 to U5, U502 to U6
