File: Hardware/Mechanical Prototype/Expansion Board/Expansion Board.kicad_pcb (KiCad board)
At the start: 2 copper layers, 100 x 70 mm, 5 parts, among them J101 Conn_02x32_Row_Letter_First, J102 Conn_01x32, J103 Conn_01x32

Commit message: 2025-03-08: Mechanical Prototype, Order #1
Parts:
- H101, H102: value M3 -> MountingBracket_612; footprint MountingHole:MountingHole_3.2mm_M3_DIN965 -> Mechanical Prototype:MountingBracket_612_M3
- moved H101 0.20 mm to (90.7, 48.5)
- moved H102 0.20 mm to (90.7, 108.5)
