File: Hardware/Mechanical Prototype/Expansion Board/Expansion Board.kicad_sch (KiCad schematic)
At the start: 5 parts, among them J101 Conn_02x32_Row_Letter_First, J102 Conn_01x32, J103 Conn_01x32

Commit message: 2025-03-08: Mechanical Prototype, Order #1
Parts:
- H101, H102: value M3 -> MountingBracket_612; footprint MountingHole:MountingHole_3.2mm_M3_DIN965 -> Mechanical Prototype:MountingBracket_612_M3; symbol Mechanical:MountingHole -> Mechanical Prototype:MountingBracket_612
Changed lines of the file:
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@@
 	)
 	(symbol
-		(lib_id "Mechanical:MountingHole")
-		(at 76.2 63.5 0)
+		(lib_id "Mechanical Prototype:MountingBracket_612")
+		(at 76.2 57.15 0)
 		(unit 1)
 		(exclude_from_sim yes)
@@
 		(dnp no)
 		(property "Reference" "H102"
-			(at 79.248 62.2299 0)
+			(at 79.248 55.8799 0)
 			(effects
 				(font
@@
 			)
 		)
-		(property "Value" "M3"
-			(at 79.248 64.7699 0)
-			(effects
-				(font
-					(size 1.27 1.27)
-				)
-				(justify left)
-			)
-		)
-		(property "Footprint" "MountingHole:MountingHole_3.2mm_M3_DIN965"
-			(at 76.2 63.5 0)
-			(effects
-				(font
-					(size 1.27 1.27)
-				)
-				(hide yes)
-			)
-		)
-		(property "Datasheet" "~"
-			(at 76.2 63.5 0)
+		(property "Value" "MountingBracket_612"
+			(at 76.2 62.992 0)
+			(effects
+				(font
+					(size 1.27 1.27)
+				)
+			)
+		)
+		(property "Footprint" "Mechanical Prototype:MountingBracket_612_M3"
+			(at 76.2 57.15 0)
+			(effects
+				(font
+					(size 1.27 1.27)
+				)
+				(hide yes)
+			)
+		)
+		(property "Datasheet" "https://www.keyelco.com/userAssets/file/M65p118.pdf"
+			(at 76.2 57.15 0)
 			(effects
 				(font
@@
 		)
 		(property "Description" "Mounting Hole without connection"
-			(at 76.2 63.5 0)
+			(at 76.2 66.675 0)
 			(effects
 				(font
@@
 	)
 	(symbol
-		(lib_id "Mechanical:MountingHole")
+		(lib_id "Mechanical Prototype:MountingBracket_612")
 		(at 76.2 69.85 0)
 		(unit 1)
@@
 		(fields_autoplaced yes)
 		(property "Reference" "H101"
-			(at 79.248 68.5799 0)
+			(at 83.82 68.1354 0)
 			(effects
 				(font
@@
 			)
 		)
-		(property "Value" "M3"
-			(at 79.248 71.1199 0)
+		(property "Value" "MountingBracket_612"
+			(at 83.82 70.6754 0)
 			(effects
 				(font
@@
 			)
 		)
-		(property "Footprint" "MountingHole:MountingHole_3.2mm_M3_DIN965"
+		(property "Footprint" "Mechanical Prototype:MountingBracket_612_M3"
 			(at 76.2 69.85 0)
 			(effects
@@
 			)
 		)
-		(property "Datasheet" "~"
+		(property "Datasheet" "https://www.keyelco.com/userAssets/file/M65p118.pdf"
 			(at 76.2 69.85 0)
 			(effects
@@
 		)
 		(property "Description" "Mounting Hole without connection"
-			(at 76.2 69.85 0)
-			(effects
-				(font
+			(at 76.2 79.375 0)
+			(effects
+				(font
