File: Hardware/Backplane.proto/Backplane.kicad_pcb (KiCad board)
At the start: 4 copper layers, 240 x 87 mm, 523 parts, among them J1 10018784-10201TLF, J1003 BM04B-SRSS-TB, J1004 BM04B-SRSS-TB, J1005 BM04B-SRSS-TB, J1006 BM04B-SRSS-TB, J1102 10018784-10201TLF, J1201 BM03B-SRSS-TB, J1402 10018784-10201TLF, J1501 BM03B-SRSS-TB, J1702 10018784-10201TLF, J1801 BM03B-SRSS-TB, J2002 BM03B-SRSS-TB, J2102 Molex 105057, J2202 Molex 105057, J2203 10018784-10201TLF, J2301 BM03B-SRSS-TB, J2502 10018784-10201TLF, J2601 BM03B-SRSS-TB, J2902 Conn_02x08_Counter_Clockwise, J402 10018784-10201TLF, J501 BM03B-SRSS-TB, J702 10018784-10201TLF, J801 BM03B-SRSS-TB, Q1004 S3134K, Q1005 S3134K, Q1101 S3134K, Q1102 GSF3407, Q1103 GSF3407, Q1104 GSF3407, Q1201 S3134K, Q1401 S3134K, Q1402 GSF3407, Q1403 GSF3407, Q1404 GSF3407, Q1501 S3134K, Q1701 S3134K, Q1702 GSF3407, Q1703 GSF3407, Q1704 GSF3407, Q1801 S3134K, Q2001 S3134K, Q2201 S3134K, Q2202 GSF3407, Q2203 GSF3407, Q2204 GSF3407, Q2301 S3134K, Q2501 S3134K, Q2502 GSF3407, Q2503 GSF3407, Q2504 GSF3407, Q2601 S3134K, Q401 S3134K, Q402 GSF3407, Q403 GSF3407, Q404 GSF3407, Q501 S3134K, Q701 S3134K, Q702 GSF3407, Q703 GSF3407, Q704 GSF3407, Q801 S3134K, SW1001 Button 12mm, U1003 CD74HC221M96, U1004 PCF8523T/1,118, U102 TCA9548APWR, U1101 NL17SZS11DFT2G-Q, U1202 CH32V003FxPx, U1203 NL17SZS11DFT2G-Q, U1401 NL17SZS11DFT2G-Q, U1502 CH32V003FxPx, U1503 NL17SZS11DFT2G-Q, U1701 NL17SZS11DFT2G-Q, U1802 CH32V003FxPx, U1803 NL17SZS11DFT2G-Q, U2001 NL17SZS11DFT2G-Q, U2004 CH32V003FxPx, U201 OSC48M-3.3I/S3-20T, U202 NL17SZS11DFT2G-Q, U203 NL17SZS11DFT2G-Q, U204 NL17SZS11DFT2G-Q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

Commit message: Simplifies schematic and lays out PCB draft 1
Parts:
- removed BT1001: Keystone 3034, Battery:BatteryHolder_Keystone_3034_1x20mm
- removed C1003, C1004: 10u, Capacitor_SMD:C_0603_1608Metric
- removed C1202, C1203, C1204, C1502, C1503, C1504, C1802, C1803, C1804, C201, C202, C203, C2302, C2303, C2304, C2602, C2603, C2604, C502, C503, C504, C802, C803, C804: 100n, Capacitor_SMD:C_0603_1608Metric
- removed C2936, C2937: 22u, Capacitor_SMD:C_0603_1608Metric
- removed D1001: Something Short-Circuit Safe, Diode_SMD:D_1206_3216Metric
- removed D1005: GREEN, LED_SMD:LED_0603_1608Metric
- removed F1101, F1102, F1103, F1401, F1402, F1403, F1701, F1702, F1703, F2101, F2201, F2202, F2203, F2204, F2501, F2502, F2503, F401, F402, F403, F701, F702, F703: SMD1206B050TF/15, Fuse:Fuse_1206_3216Metric
- removed F2901, F2902, F2903: 0ZCF0400FF2A, Home Computer:FUSER_0ZCF0400FF2A
- removed J1003, J1004, J1005, J1006: BM04B-SRSS-TB, Connector_JST:JST_SH_BM04B-SRSS-TB_1x04-1MP_P1.00mm_Vertical
- removed J1201, J1501, J1801, J2002, J2301, J2601, J501, J801: BM03B-SRSS-TB, Connector_JST:JST_SH_BM03B-SRSS-TB_1x03-1MP_P1.00mm_Vertical
- removed J2102, J2202: Molex 105057, Connector_USB:USB_A_Molex_105057_Vertical
- removed J2902: Conn_02x08_Counter_Clockwise, Connector_PinHeader_2.54mm:PinHeader_2x08_P2.54mm_Vertical_SMD
- removed Q1004, Q1005, Q1101, Q1201, Q1401, Q1501, Q1701, Q1801, Q2001, Q2201, Q2301, Q2501, Q2601, Q401, Q501, Q701, Q801: S3134K, Package_TO_SOT_SMD:SOT-23
- removed Q1102, Q1103, Q1104, Q1402, Q1403, Q1404, Q1702, Q1703, Q1704, Q2202, Q2203, Q2204, Q2502, Q2503, Q2504, Q402, Q403, Q404, Q702, Q703, Q704: GSF3407, Package_TO_SOT_SMD:SOT-23
- removed R1006, R1008, R1011, R1108, R1113, R1208, R1210, R1408, R1413, R1508, R1510, R1708, R1713, R1808, R1810, R2002, R2004, R2210, R2215, R2308, R2310, R2508, R2513, R2608, R2610, R408, R413, R508, R510, R708, R713, R808, R810: 560, Resistor_SMD:R_0603_1608Metric
- removed R1009, R1010, R1013, R1014, R1015, R1016, R1107, R1111, R1201, R1209, R1407, R1411, R1501, R1509, R1707, R1711, R1801, R1809, R2001, R2003, R2209, R2213, R2301, R2309, R2507, R2511, R2601, R2609, R407, R411, R501, R509, R707, R711, R801, R809: 10K, Resistor_SMD:R_0603_1608Metric
- removed R1202, R1502, R1802, R214, R2302, R2602, R502, R802: 6K8 1%, Resistor_SMD:R_0603_1608Metric
- removed R1203, R1204, R1205, R1207, R1503, R1504, R1505, R1507, R1803, R1804, R1805, R1807, R215, R216, R217, R219, R2303, R2304, R2305, R2307, R2603, R2604, R2605, R2607, R503, R504, R505, R507, R803, R804, R805, R807: 1K8 1%, Resistor_SMD:R_0603_1608Metric
- removed R1206, R1506, R1806, R218, R2306, R2606, R506, R806: 560 1%, Resistor_SMD:R_0603_1608Metric
- removed R2102, R2103, R2202, R2203: 0, Resistor_SMD:R_0603_1608Metric
- removed TP1001, TP1004, TP1005, TP1006, TP1007, TP1008, TP1009, TP1010, TP1101, TP1102, TP1103, TP1201, TP1202, TP1401, TP1402, TP1403, TP1501, TP1502, TP1701, TP1702, TP1703, TP1801, TP1802, TP2003, TP2004, TP2005, TP2006, TP2007, TP2008, TP2009, TP2010, TP2011, TP2012, TP2013, TP2014, TP2015, TP2016, TP2017, TP2018, TP2019, TP2020, TP2021, TP2022, TP2023, TP2024, TP2025, TP2026, TP2027, TP2028, TP2103, TP2104, TP2105, TP2201, TP2202, TP2203, TP2204, TP2205, TP2206, TP2301, TP2302, TP2501, TP2502, TP2503, TP2601, TP2602, TP401, TP402, TP403, TP501, TP502, TP701, TP702, TP703, TP801, TP802: TestPoint_Small, TestPoint:TestPoint_Pad_D1.0mm
- removed TP2901: +12V, TestPoint:TestPoint_Pad_D2.0mm
- removed TP2902: +5V, TestPoint:TestPoint_Pad_D2.0mm
- removed TP2903: +3V3, TestPoint:TestPoint_Pad_D2.0mm
- removed TP2904, TP2905: +1V8, TestPoint:TestPoint_Pad_D2.0mm
- removed U1003: CD74HC221M96, Package_SO:SOIC-16_3.9x9.9mm_P1.27mm
- removed U1004: PCF8523T/1,118, Home Computer:PCF8523T1,118
- removed U1101, U1203, U1401, U1503, U1701, U1803, U2001, U202, U204, U205, U2201, U2303, U2501, U2603, U401, U503, U701, U803: NL17SZS11DFT2G-Q, Package_TO_SOT_SMD:SOT-363_SC-70-6
- removed Y1001: 32.768k, Crystal:Crystal_SMD_3215-2Pin_3.2x1.5mm
- added C2938: 22u, Capacitor_SMD:CP_Elec_4x5.4, B.Cu at (130.8, 72.6)
- added C2939: 22u, Capacitor_SMD:CP_Elec_4x5.4, B.Cu at (125.8, 72.6)
- added J10: Conn_01x03, Connector_PinHeader_2.54mm:PinHeader_1x03_P2.54mm_Vertical, B.Cu at (210.0, 116.3)
- added J11: Conn_01x03, Connector_PinHeader_2.54mm:PinHeader_1x03_P2.54mm_Vertical, B.Cu at (190.4, 84.7)
- added J12: Conn_01x03, Connector_PinHeader_2.54mm:PinHeader_1x03_P2.54mm_Vertical, B.Cu at (238.0, 116.3)
- added J13: Conn_01x03, Connector_PinHeader_2.54mm:PinHeader_1x03_P2.54mm_Vertical, B.Cu at (266.0, 116.3)
- added J14: Conn_01x06, Connector_PinHeader_2.54mm:PinHeader_1x06_P2.54mm_Vertical, B.Cu at (35.5, 128.2)
- added J15: Conn_02x03_Odd_Even, Connector_PinHeader_2.54mm:PinHeader_2x03_P2.54mm_Vertical, F.Cu at (84.5, 131.6)
- added J16: Conn_02x03_Odd_Even, Connector_PinHeader_2.54mm:PinHeader_2x03_P2.54mm_Vertical, F.Cu at (112.5, 131.6)
- added J17: Conn_02x03_Odd_Even, Connector_PinHeader_2.54mm:PinHeader_2x03_P2.54mm_Vertical, F.Cu at (140.5, 131.6)
- added J18: Conn_02x03_Odd_Even, Connector_PinHeader_2.54mm:PinHeader_2x03_P2.54mm_Vertical, F.Cu at (168.5, 131.6)
- added J19: Conn_02x03_Odd_Even, Connector_PinHeader_2.54mm:PinHeader_2x03_P2.54mm_Vertical, F.Cu at (196.5, 131.6)
- added J2: ~, Connector_PinHeader_2.54mm:PinHeader_1x04_P2.54mm_Vertical, F.Cu at (70.6, 95.3)
- added J20: Conn_02x03_Odd_Even, Connector_PinHeader_2.54mm:PinHeader_2x03_P2.54mm_Vertical, F.Cu at (224.5, 131.6)
- added J21: Conn_02x03_Odd_Even, Connector_PinHeader_2.54mm:PinHeader_2x03_P2.54mm_Vertical, F.Cu at (252.5, 131.6)
- added J3: ~, Connector_PinHeader_2.54mm:PinHeader_1x04_P2.54mm_Vertical, F.Cu at (66.8, 95.3)
- added J4: ~, Connector_PinHeader_2.54mm:PinHeader_1x04_P2.54mm_Vertical, B.Cu at (189.3, 89.2)
- added J5: ~, Connector_PinHeader_2.54mm:PinHeader_1x04_P2.54mm_Vertical, B.Cu at (106.2, 72.3)
- added J6: Conn_01x03, Connector_PinHeader_2.54mm:PinHeader_1x03_P2.54mm_Vertical, B.Cu at (98.0, 116.3)
- added J7: Conn_01x03, Connector_PinHeader_2.54mm:PinHeader_1x03_P2.54mm_Vertical, B.Cu at (126.0, 116.3)
- added J8: Conn_01x03, Connector_PinHeader_2.54mm:PinHeader_1x03_P2.54mm_Vertical, B.Cu at (154.0, 116.3)
- added J9: Conn_01x03, Connector_PinHeader_2.54mm:PinHeader_1x03_P2.54mm_Vertical, B.Cu at (182.0, 116.3)
- added JP1: Jumper_2_Bridged, Connector_PinHeader_2.54mm:PinHeader_1x02_P2.54mm_Vertical, B.Cu at (155.1, 90.9)
- added R3003: 560, Resistor_SMD:R_0603_1608Metric, B.Cu at (157.7, 101.0)
- added TP409: TestPoint_Small, TestPoint:TestPoint_Pad_D1.0mm, B.Cu at (162.3, 89.2)
- added TP410: TestPoint_Small, TestPoint:TestPoint_Pad_D1.0mm, B.Cu at (163.1, 97.4)
- C2901: footprint Capacitor_SMD:C_1206_3216Metric -> Capacitor_SMD:CP_Elec_6.3x9.9
- NT2906: moved to F.Cu
- TP2906: footprint Jumper:SolderJumper-2_P1.3mm_Open_Pad1.0x1.5mm -> Connector_PinHeader_2.54mm:PinHeader_1x02_P2.54mm_Vertical
- moved SW1001 230.0 mm to (35.7, 113.3), turned to -90 degrees
- moved R1003 217.4 mm to (38.9, 119.0), turned to 90 degrees
- moved R1007 200.7 mm to (191.8, 92.0)
- moved D1004 195.0 mm to (192.2, 89.5), turned to -90 degrees
- moved R1005 194.6 mm to (184.1, 101.4), turned to 0 degrees
- moved D1003 191.3 mm to (184.1, 103.0)
- moved C2002 180.6 mm to (182.0, 96.3), turned to -90 degrees
- moved U2004 158.4 mm to (186.5, 96.3), turned to 90 degrees
- moved R3002 158.1 mm to (160.3, 91.1), turned to -90 degrees
- moved U203 156.3 mm to (163.3, 94.3), turned to 90 degrees
- moved R203 154.8 mm to (165.4, 92.5), turned to 90 degrees
- moved U3002 153.6 mm to (158.3, 91.0), turned to 90 degrees
- moved C205 148.0 mm to (159.1, 93.8)
- moved C204 148.0 mm to (159.1, 99.2)
- moved R201 144.6 mm to (155.6, 95.3), turned to -90 degrees
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Connections:
- C101 pad 2: +3V3 -> +1V8
- C2901 pad 1: GND -> +5V
- C2901 pad 2: +5V -> GND
- J1 pad B13: unconnected-(J1-GP0-PadB13) -> /FAB_{0}
- J1 pad B14: unconnected-(J1-GP1-PadB14) -> /FAB_{1}
- J1 pad B16: unconnected-(J1-GP2-PadB16) -> /FAB_{2}
- J1 pad B17: unconnected-(J1-GP3-PadB17) -> /FAB_{3}
- J1 pad B19: unconnected-(J1-GP4-PadB19) -> /FAB_{4}
- J1 pad B20: unconnected-(J1-GP5-PadB20) -> /FAB_{5}
- J1 pad B22: unconnected-(J1-GP6-PadB22) -> /FAB_{6}
- J1 pad B23: unconnected-(J1-GP7-PadB23) -> /FAB_{7}
- R1003 pad 1: +3V3 -> ~{RESET}
- R1003 pad 2: ~{RESET} -> +3V3
- U102 pad 13: /Expansions/I2C4_{SDA} -> /Expansions/I2C2_{SDA}
- U102 pad 14: /Expansions/I2C4_{SCL} -> /Expansions/I2C2_{SCL}
- U102 pad 15: /Expansions/I2C5_{SDA} -> /Expansions/I2C1_{SDA}
- U102 pad 16: /Expansions/I2C5_{SCL} -> /Expansions/I2C1_{SCL}
- U102 pad 17: /Expansions/I2C6_{SDA} -> /Expansions/I2C0_{SDA}
- U102 pad 18: /Expansions/I2C6_{SCL} -> /Expansions/I2C0_{SCL}
- U102 pad 24: +5V -> +1V8
- U102 pad 3: ~{RESET} -> /Builtins/~{RESET_I2C}
- U102 pad 4: /Expansions/I2C0_{SCL} -> /Expansions/I2C6_{SDA}
- U102 pad 5: /Expansions/I2C0_{SDA} -> /Expansions/I2C6_{SCL}
- U102 pad 6: /Expansions/I2C1_{SDA} -> /Expansions/I2C5_{SDA}
- U102 pad 7: /Expansions/I2C1_{SCL} -> /Expansions/I2C5_{SCL}
- U102 pad 8: /Expansions/I2C2_{SDA} -> /Expansions/I2C4_{SDA}
- U102 pad 9: /Expansions/I2C2_{SCL} -> /Expansions/I2C4_{SCL}
- U1202 pad 1: /Expansions/Module Slot 2/Management Controller/MEAS_+12V -> unconnected-(U1202-PD4-Pad1)
- U1202 pad 15: Net-(U1202-PC5) -> /Expansions/Module Slot 2/~{CARD_RESET}
- U1202 pad 19: /Expansions/Module Slot 2/~{MOD_CLK_EN} -> /Expansions/Module Slot 2/Management Controller/OUT1
- U1202 pad 2: /Expansions/Module Slot 2/Management Controller/MEAS_+5V -> unconnected-(U1202-PD5-Pad2)
- U1202 pad 3: /Expansions/Module Slot 2/Management Controller/MEAS_+3V3 -> unconnected-(U1202-PD6-Pad3)
- U1202 pad 4: /Expansions/Module Slot 2/Management Controller/MGMT_~{RST} -> ~{RESET}
- U1202 pad 8: /Expansions/Module Slot 2/POWER_ON -> /Expansions/Module Slot 2/Management Controller/OUT0
- U1502 pad 1: /Expansions/Module Slot 3/Management Controller/MEAS_+12V -> unconnected-(U1502-PD4-Pad1)
- U1502 pad 15: Net-(U1502-PC5) -> /Expansions/Module Slot 3/~{CARD_RESET}
- U1502 pad 19: /Expansions/Module Slot 3/~{MOD_CLK_EN} -> /Expansions/Module Slot 3/Management Controller/OUT1
- U1502 pad 2: /Expansions/Module Slot 3/Management Controller/MEAS_+5V -> unconnected-(U1502-PD5-Pad2)
- U1502 pad 3: /Expansions/Module Slot 3/Management Controller/MEAS_+3V3 -> unconnected-(U1502-PD6-Pad3)
- U1502 pad 4: /Expansions/Module Slot 3/Management Controller/MGMT_~{RST} -> ~{RESET}
- U1502 pad 8: /Expansions/Module Slot 3/POWER_ON -> /Expansions/Module Slot 3/Management Controller/OUT0
- U1802 pad 1: /Expansions/Module Slot 4/Management Controller/MEAS_+12V -> unconnected-(U1802-PD4-Pad1)
- U1802 pad 15: Net-(U1802-PC5) -> /Expansions/Module Slot 4/~{CARD_RESET}
- U1802 pad 19: /Expansions/Module Slot 4/~{MOD_CLK_EN} -> /Expansions/Module Slot 4/Management Controller/OUT1
- U1802 pad 2: /Expansions/Module Slot 4/Management Controller/MEAS_+5V -> unconnected-(U1802-PD5-Pad2)
- U1802 pad 3: /Expansions/Module Slot 4/Management Controller/MEAS_+3V3 -> unconnected-(U1802-PD6-Pad3)
- U1802 pad 4: /Expansions/Module Slot 4/Management Controller/MGMT_~{RST} -> ~{RESET}
- U1802 pad 8: /Expansions/Module Slot 4/POWER_ON -> /Expansions/Module Slot 4/Management Controller/OUT0
- U2004 pad 1: /Builtins/Management Controller/MEAS_+12V -> unconnected-(U2004-PD4-Pad1)
- U2004 pad 15: Net-(U2004-PC5) -> ~{RESET}
- U2004 pad 2: /Builtins/Management Controller/MEAS_+5V -> unconnected-(U2004-PD5-Pad2)
- U2004 pad 20: /Builtins/BRD_LED2 -> /Builtins/~{RESET_I2C}
- U2004 pad 3: /Builtins/Management Controller/MEAS_+3V3 -> unconnected-(U2004-PD6-Pad3)
- U2004 pad 4: /Builtins/Management Controller/MGMT_~{RST} -> ~{RESET}
- U203 pad 4: /Expansions/Clock/CLK_SPAN -> /Expansions/CLKTREE_{2}
- U2302 pad 1: /Expansions/Module Slot 5/Management Controller/MEAS_+12V -> unconnected-(U2302-PD4-Pad1)
- U2302 pad 15: Net-(U2302-PC5) -> /Expansions/Module Slot 5/~{CARD_RESET}
- U2302 pad 19: /Expansions/Module Slot 5/~{MOD_CLK_EN} -> /Expansions/Module Slot 5/Management Controller/OUT1
- U2302 pad 2: /Expansions/Module Slot 5/Management Controller/MEAS_+5V -> unconnected-(U2302-PD5-Pad2)
- U2302 pad 3: /Expansions/Module Slot 5/Management Controller/MEAS_+3V3 -> unconnected-(U2302-PD6-Pad3)
- U2302 pad 4: /Expansions/Module Slot 5/Management Controller/MGMT_~{RST} -> ~{RESET}
- U2302 pad 8: /Expansions/Module Slot 5/POWER_ON -> /Expansions/Module Slot 5/Management Controller/OUT0
- U2602 pad 1: /Expansions/Module Slot 6/Management Controller/MEAS_+12V -> unconnected-(U2602-PD4-Pad1)
- U2602 pad 15: Net-(U2602-PC5) -> /Expansions/Module Slot 6/~{CARD_RESET}
- U2602 pad 19: /Expansions/Module Slot 6/~{MOD_CLK_EN} -> /Expansions/Module Slot 6/Management Controller/OUT1
- U2602 pad 2: /Expansions/Module Slot 6/Management Controller/MEAS_+5V -> unconnected-(U2602-PD5-Pad2)
- U2602 pad 3: /Expansions/Module Slot 6/Management Controller/MEAS_+3V3 -> unconnected-(U2602-PD6-Pad3)
- U2602 pad 4: /Expansions/Module Slot 6/Management Controller/MGMT_~{RST} -> ~{RESET}
- U2602 pad 8: /Expansions/Module Slot 6/POWER_ON -> /Expansions/Module Slot 6/Management Controller/OUT0
- U2901 pad 10: /Expansions/MOD0_{GP5} -> /Expansions/MOD6_{GP5}
- U2901 pad 12: /Expansions/MOD0_{GP6} -> /Expansions/MOD6_{GP6}
- U2901 pad 13: /Expansions/MOD0_{GP7} -> /Expansions/MOD6_{GP7}
- U2901 pad 15: /Expansions/MOD1_{GP0} -> /Expansions/MOD5_{GP0}
- U2901 pad 16: /Expansions/MOD1_{GP1} -> /Expansions/MOD5_{GP1}
- U2901 pad 18: /Expansions/MOD1_{GP2} -> /Expansions/MOD5_{GP2}
- U2901 pad 19: /Expansions/MOD1_{GP3} -> /Expansions/MOD5_{GP3}
- U2901 pad 21: /Expansions/MOD1_{GP4} -> /Expansions/MOD5_{GP4}
- U2901 pad 22: /Expansions/MOD1_{GP5} -> /Expansions/MOD5_{GP5}
- U2901 pad 24: /Expansions/MOD1_{GP6} -> /Expansions/MOD5_{GP6}
- U2901 pad 25: /Expansions/MOD1_{GP7} -> /Expansions/MOD5_{GP7}
- U2901 pad 27: /Expansions/MOD2_{GP0} -> /Expansions/MOD4_{GP0}
- U2901 pad 28: /Expansions/MOD2_{GP1} -> /Expansions/MOD4_{GP1}
- U2901 pad 3: /Expansions/MOD0_{GP0} -> /Expansions/MOD6_{GP0}
- U2901 pad 30: /Expansions/MOD2_{GP2} -> /Expansions/MOD4_{GP2}
- U2901 pad 31: /Expansions/MOD2_{GP3} -> /Expansions/MOD4_{GP3}
- U2901 pad 33: /Expansions/MOD2_{GP4} -> /Expansions/MOD4_{GP4}
- U2901 pad 34: /Expansions/MOD2_{GP5} -> /Expansions/MOD4_{GP5}
- U2901 pad 36: /Expansions/MOD2_{GP6} -> /Expansions/MOD4_{GP6}
- U2901 pad 37: /Expansions/MOD2_{GP7} -> /Expansions/MOD4_{GP7}
- U2901 pad 4: /Expansions/MOD0_{GP1} -> /Expansions/MOD6_{GP1}
- U2901 pad 53: /Expansions/MOD4_{GP0} -> /Expansions/MOD2_{GP0}
- U2901 pad 54: /Expansions/MOD4_{GP1} -> /Expansions/MOD2_{GP1}
- U2901 pad 56: /Expansions/MOD4_{GP2} -> /Expansions/MOD2_{GP2}
- U2901 pad 57: /Expansions/MOD4_{GP3} -> /Expansions/MOD2_{GP3}
- U2901 pad 59: /Expansions/MOD4_{GP4} -> /Expansions/MOD2_{GP4}
- U2901 pad 6: /Expansions/MOD0_{GP2} -> /Expansions/MOD6_{GP2}
- U2901 pad 60: /Expansions/MOD4_{GP5} -> /Expansions/MOD2_{GP5}
- U2901 pad 62: /Expansions/MOD4_{GP6} -> /Expansions/MOD2_{GP6}
- U2901 pad 63: /Expansions/MOD4_{GP7} -> /Expansions/MOD2_{GP7}
- U2901 pad 65: /Expansions/MOD5_{GP0} -> /Expansions/MOD1_{GP0}
- U2901 pad 66: /Expansions/MOD5_{GP1} -> /Expansions/MOD1_{GP1}
- U2901 pad 68: /Expansions/MOD5_{GP2} -> /Expansions/MOD1_{GP2}
- U2901 pad 69: /Expansions/MOD5_{GP3} -> /Expansions/MOD1_{GP3}
- U2901 pad 7: /Expansions/MOD0_{GP3} -> /Expansions/MOD6_{GP3}
- U2901 pad 71: /Expansions/MOD5_{GP4} -> /Expansions/MOD1_{GP4}
- U2901 pad 72: /Expansions/MOD5_{GP5} -> /Expansions/MOD1_{GP5}
- U2901 pad 74: /Expansions/MOD5_{GP6} -> /Expansions/MOD1_{GP6}
- U2901 pad 75: /Expansions/MOD5_{GP7} -> /Expansions/MOD1_{GP7}
- U2901 pad 77: /Expansions/MOD6_{GP0} -> /Expansions/MOD0_{GP0}
- U2901 pad 78: /Expansions/MOD6_{GP1} -> /Expansions/MOD0_{GP1}
- U2901 pad 80: /Expansions/MOD6_{GP2} -> /Expansions/MOD0_{GP2}
- U2901 pad 81: /Expansions/MOD6_{GP3} -> /Expansions/MOD0_{GP3}
- U2901 pad 83: /Expansions/MOD6_{GP4} -> /Expansions/MOD0_{GP4}
- U2901 pad 84: /Expansions/MOD6_{GP5} -> /Expansions/MOD0_{GP5}
- U2901 pad 86: /Expansions/MOD6_{GP6} -> /Expansions/MOD0_{GP6}
- U2901 pad 87: /Expansions/MOD6_{GP7} -> /Expansions/MOD0_{GP7}
- U2901 pad 89: /Expansions/FAB_{0} -> /FAB_{0}
- U2901 pad 9: /Expansions/MOD0_{GP4} -> /Expansions/MOD6_{GP4}
- U2901 pad 90: /Expansions/FAB_{1} -> /FAB_{1}
- U2901 pad 92: /Expansions/FAB_{2} -> /FAB_{2}
- U2901 pad 93: /Expansions/FAB_{3} -> /FAB_{3}
- U2901 pad 95: /Expansions/FAB_{4} -> /FAB_{4}
- U2901 pad 96: /Expansions/FAB_{5} -> /FAB_{5}
- U2901 pad 98: /Expansions/FAB_{6} -> /FAB_{6}
- U2901 pad 99: /Expansions/FAB_{7} -> /FAB_{7}
- U3002 pad 4: /Expansions/P2_CLK -> Net-(JP1-A)
- U502 pad 1: /Expansions/Module Slot 0/Management Controller/MEAS_+12V -> unconnected-(U502-PD4-Pad1)
- U502 pad 15: Net-(U502-PC5) -> /Expansions/Module Slot 0/~{CARD_RESET}
- U502 pad 19: /Expansions/Module Slot 0/~{MOD_CLK_EN} -> /Expansions/Module Slot 0/Management Controller/OUT1
- U502 pad 2: /Expansions/Module Slot 0/Management Controller/MEAS_+5V -> unconnected-(U502-PD5-Pad2)
- U502 pad 3: /Expansions/Module Slot 0/Management Controller/MEAS_+3V3 -> unconnected-(U502-PD6-Pad3)
- U502 pad 4: /Expansions/Module Slot 0/Management Controller/MGMT_~{RST} -> ~{RESET}
- U502 pad 8: /Expansions/Module Slot 0/POWER_ON -> /Expansions/Module Slot 0/Management Controller/OUT0
- U802 pad 1: /Expansions/Module Slot 1/Management Controller/MEAS_+12V -> unconnected-(U802-PD4-Pad1)
- U802 pad 15: Net-(U802-PC5) -> /Expansions/Module Slot 1/~{CARD_RESET}
- U802 pad 19: /Expansions/Module Slot 1/~{MOD_CLK_EN} -> /Expansions/Module Slot 1/Management Controller/OUT1
- U802 pad 2: /Expansions/Module Slot 1/Management Controller/MEAS_+5V -> unconnected-(U802-PD5-Pad2)
- U802 pad 3: /Expansions/Module Slot 1/Management Controller/MEAS_+3V3 -> unconnected-(U802-PD6-Pad3)
- U802 pad 4: /Expansions/Module Slot 1/Management Controller/MGMT_~{RST} -> ~{RESET}
- U802 pad 8: /Expansions/Module Slot 1/POWER_ON -> /Expansions/Module Slot 1/Management Controller/OUT0
Routing:
- net ~{RESET}: track 0.00 -> 425.1 mm, vias 0 -> 8
- net +1V8: track 0.00 -> 337.5 mm, vias 0 -> 33
- net I2C^{BRD}_{SCL}: track 29.0 -> 272.6 mm, vias 0 -> 10
- net I2C^{BRD}_{SDA}: track 26.3 -> 266.4 mm, vias 0 -> 10
- net +3V3: track 23.1 -> 231.7 mm, vias 4 -> 58
- net /Expansions/CLKTREE_{2}: track 0.00 -> 163.9 mm, vias 0 -> 2
- net +5V: track 2.25 -> 164.7 mm, vias 1 -> 4
- net /Expansions/FAB_~{RES}: track 0.00 -> 152.4 mm
- net /Expansions/MOD6_{GP0}: track 0.00 -> 146.3 mm
- net /Expansions/MOD6_{GP1}: track 0.00 -> 142.4 mm
- net /Expansions/MOD6_{GP2}: track 0.00 -> 139.2 mm
- net /Expansions/MOD6_{GP3}: track 0.00 -> 139.2 mm
- net /Expansions/MOD6_{GP4}: track 0.00 -> 136.1 mm
- net /Expansions/MOD6_{GP5}: track 0.00 -> 132.1 mm
- net /Expansions/MOD6_{GP7}: track 0.00 -> 129.0 mm
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- added copper zone on In2.Cu, net GND
- removed copper zone on In2.Cu, net +5V
