File: Hardware/Backplane.proto/Backplane.kicad_pcb (KiCad board)
At the start: 4 copper layers, 240 x 87 mm, 217 parts, among them J1 10018784-10201TLF, J10 Conn_01x03, J11 Conn_01x03, J1102 10018784-10201TLF, J12 Conn_01x03, J13 Conn_01x03, J14 Conn_01x06, J1402 10018784-10201TLF, J15 Conn_02x03_Odd_Even, J16 Conn_02x03_Odd_Even, J17 Conn_02x03_Odd_Even, J1702 10018784-10201TLF, J18 Conn_02x03_Odd_Even, J19 Conn_02x03_Odd_Even, J20 Conn_02x03_Odd_Even, J21 Conn_02x03_Odd_Even, J2203 10018784-10201TLF, J2502 10018784-10201TLF, J402 10018784-10201TLF, J6 Conn_01x03, J7 Conn_01x03, J702 10018784-10201TLF, J8 Conn_01x03, J9 Conn_01x03, SW1001 Button 12mm, U102 TCA9548APWR, U1202 CH32V003FxPx, U1502 CH32V003FxPx, U1802 CH32V003FxPx, U2004 CH32V003FxPx, U201 OSC48M-3.3I/S3-20T, U203 NL17SZS11DFT2G-Q, U2302 CH32V003FxPx, U2602 CH32V003FxPx, U2901 P2X8C4M64P, U2902 AP3445LW6-7, U3001 NL17SZS11DFT2G-Q, U3002 NL17SZS11DFT2G-Q, U502 CH32V003FxPx, U802 CH32V003FxPx

Commit message: Adds huge TODO so i don't forget to do the silkscreen.
Other:
- board text added: "TODO!"
