File: Hardware/Backplane.proto/Backplane.kicad_sch (KiCad schematic)
At the start: 9 parts, among them J1 10018784-10201TLF

Commit message: Simplifies schematic and lays out PCB draft 1
Connections:
- net FAB_{0}: now reaches J1.B13 (GP0)
- net FAB_{1}: now reaches J1.B14 (GP1)
- net FAB_{2}: now reaches J1.B16 (GP2)
- net FAB_{3}: now reaches J1.B17 (GP3)
- net FAB_{4}: now reaches J1.B19 (GP4)
- net FAB_{5}: now reaches J1.B20 (GP5)
- net FAB_{6}: now reaches J1.B22 (GP6)
- net FAB_{7}: now reaches J1.B23 (GP7)
Changed lines of the file:
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@@
+		)
+	)
+	(label "FAB_{5}"
+		(at 81.915 139.7 180)
+		(effects
+			(font
+				(size 1.016 1.016)
+			)
+			(justify right bottom)
 		)
 	)
@@
 		)
 	)
+	(label "FAB_{5}"
+		(at 168.275 83.185 180)
+		(effects
+			(font
+				(size 1.016 1.016)
+			)
+			(justify right bottom)
+		)
+	)
 	(label "I2C^{FAB}_{SCL}"
 		(at 111.125 45.085 180)
@@
 		)
 	)
+	(label "FAB_{3}"
+		(at 81.915 134.62 180)
+		(effects
+			(font
+				(size 1.016 1.016)
+			)
+			(justify right bottom)
+		)
+	)
+	(label "FAB_{6}"
+		(at 81.915 142.24 180)
+		(effects
+			(font
+				(size 1.016 1.016)
+			)
+			(justify right bottom)
+		)
+	)
 	(label "USB_{1}_D-"
 		(at 221.615 114.3 0)
@@
 		)
 	)
+	(label "FAB_{3}"
+		(at 168.275 75.565 180)
+		(effects
+			(font
+				(size 1.016 1.016)
+			)
+			(justify right bottom)
+		)
+	)
 	(label "USB_{1}_D+"
 		(at 221.615 111.76 0)
@@
 		)
 	)
+	(label "FAB_{6}"
+		(at 168.275 88.265 180)
+		(effects
+			(font
+				(size 1.016 1.016)
+			)
+			(justify right bottom)
+		)
+	)
+	(label "FAB_{1}"
+		(at 81.9228 129.54 180)
+		(effects
+			(font
+				(size 1.016 1.016)
+			)
+			(justify right bottom)
+		)
+	)
+	(label "FAB_{4}"
+		(at 168.275 80.645 180)
+		(effects
+			(font
+				(size 1.016 1.016)
+			)
+			(justify right bottom)
+		)
+	)
+	(label "FAB_{0}"
+		(at 168.275 65.405 180)
+		(effects
+			(font
+				(size 1.016 1.016)
+			)
+			(justify right bottom)
+		)
+	)
+	(label "FAB_{7}"
+		(at 168.275 90.805 180)
+		(effects
+			(font
+				(size 1.016 1.016)
+			)
+			(justify right bottom)
+		)
+	)
 	(label "USB_{0}_D-"
 		(at 221.615 98.425 0)
@@
 		)
 	)
+	(label "FAB_{4}"
+		(at 81.915 137.16 180)
+		(effects
+			(font
+				(size 1.016 1.016)
+			)
+			(justify right bottom)
+		)
+	)
+	(label "FAB_{2}"
+		(at 81.915 132.08 180)
+		(effects
+			(font
+				(size 1.016 1.016)
+			)
+			(justify right bottom)
+		)
+	)
+	(label "FAB_{0}"
+		(at 81.915 127 180)
+		(effects
+			(font
+				(size 1.016 1.016)
+			)
+			(justify right bottom)
+		)
+	)
+	(label "FAB_{2}"
+		(at 168.275 73.025 180)
+		(effects
+			(font
+				(size 1.016 1.016)
+			)
+			(justify right bottom)
+		)
+	)
+	(label "FAB_{7}"
+		(at 81.915 144.78 180)
+		(effects
+			(font
+				(size 1.016 1.016)
+			)
+			(justify right bottom)
+		)
+	)
+	(label "FAB_{1}"
+		(at 168.275 67.945 180)
+		(effects
+			(font
+				(size 1.016 1.016)
+			)
+			(justify right bottom)
+		)
+	)
