File: Hardware/Backplane.proto/builtins.kicad_sch (KiCad schematic)
At the start: 37 parts, among them J1003 BM04B-SRSS-TB, J1004 BM04B-SRSS-TB, J1005 BM04B-SRSS-TB, J1006 BM04B-SRSS-TB, Q1004 S3134K, Q1005 S3134K, SW1001 Button 12mm, U1003 CD74HC221M96, U1004 PCF8523T/1,118, Y1001 32.768k

Commit message: Simplifies schematic and lays out PCB draft 1
Parts:
- removed BT1001: Keystone 3034, Battery:BatteryHolder_Keystone_3034_1x20mm, symbol Device:Battery_Cell
- removed C1003, C1004: 10u, Capacitor_SMD:C_0603_1608Metric, symbol Device:C_Small
- removed D1001: Something Short-Circuit Safe, Diode_SMD:D_1206_3216Metric, symbol Device:D_Small
- removed J1003, J1004, J1005, J1006: BM04B-SRSS-TB, Connector_JST:JST_SH_BM04B-SRSS-TB_1x04-1MP_P1.00mm_Vertical, symbol Connector_Generic:Conn_01x04
- removed Q1004, Q1005: S3134K, Package_TO_SOT_SMD:SOT-23, symbol Home Computer:S3134K
- removed R1006, R1011: 560, Resistor_SMD:R_0603_1608Metric, symbol Device:R
- removed R1009, R1010, R1013, R1014, R1015, R1016: 10K, Resistor_SMD:R_0603_1608Metric, symbol Device:R
- removed TP1001, TP1004, TP1005, TP1006, TP1007, TP1008, TP1009, TP1010: TestPoint_Small, TestPoint:TestPoint_Pad_D1.0mm, symbol Connector:TestPoint_Small
- removed U1003: CD74HC221M96, Package_SO:SOIC-16_3.9x9.9mm_P1.27mm, symbol Symbol Library:CD74HC221M96
- removed U1004: PCF8523T/1,118, Home Computer:PCF8523T1,118, symbol Home Computer:PCF8523T/1
- removed Y1001: 32.768k, Crystal:Crystal_SMD_3215-2Pin_3.2x1.5mm, symbol Device:Crystal
- added J4, J5: (no value), Connector_PinHeader_2.54mm:PinHeader_1x04_P2.54mm_Vertical, symbol Connector_Generic:Conn_01x04
- SW1001: now fitted
Connections:
- net +3V3: now also R1003.2, J4.1 (Pin_1), J5.1 (Pin_1); no longer R1003.1
- net GND: now also J4.4 (Pin_4), J5.4 (Pin_4)
- net I2C^{BRD}_{SCL}: now also J4.2 (Pin_2)
- net I2C^{BRD}_{SDA}: now also J4.3 (Pin_3)
- net POWER_OK: now also J5.3 (Pin_3)
- net ~{RESET}: now also R1003.1, J5.2 (Pin_2); no longer R1003.2
- no-connect marks 5 -> 3
Other:
- sheet Management Controller ports: added none; removed REF_+12V, REF_+3V3, REF_+5V
- note removed: "Test point for trimming"
- note removed: "This should be in the "unreset" state, as we do want the system to power up"
- moved on the sheet: R1003
