File: Hardware/Backplane.proto/clock.kicad_sch (KiCad schematic)
At the start: 10 parts, among them U201 OSC48M-3.3I/S3-20T, U202 NL17SZS11DFT2G-Q, U203 NL17SZS11DFT2G-Q, U204 NL17SZS11DFT2G-Q, U205 NL17SZS11DFT2G-Q

Commit message: Simplifies schematic and lays out PCB draft 1
Parts:
- removed U202, U204, U205: NL17SZS11DFT2G-Q, Package_TO_SOT_SMD:SOT-363_SC-70-6, symbol Home Computer:NL17SZS11DFT2G-Q
- added TP409, TP410: TestPoint_Small, TestPoint:TestPoint_Pad_D1.0mm, symbol Connector:TestPoint_Small
Connections:
- net CLK_SPAN is gone; now on net CLKTREE2: U203.4 (Y)
- net CLKTREE2: now also TP409.1
- net CLK_RAW: now also TP410.1
