File: Hardware/Backplane.proto/expansions.kicad_sch (KiCad schematic)
At the start: 9 parts, among them U102 TCA9548APWR, U2901 P2X8C4M64P, U3001 NL17SZS11DFT2G-Q, U3002 NL17SZS11DFT2G-Q

Commit message: Simplifies schematic and lays out PCB draft 1
Parts:
- added JP1: Jumper_2_Bridged, Connector_PinHeader_2.54mm:PinHeader_1x02_P2.54mm_Vertical, symbol Jumper:Jumper_2_Bridged
Connections:
- net +1V8: now also C101.2
- net +3V3: no longer C101.2
- net I2C0_{SCL}: now also U102.18 (SC6); no longer U102.4 (SD0)
- net I2C0_{SDA}: now also U102.17 (SD6); no longer U102.5 (SC0)
- net I2C1_{SCL}: now also U102.16 (SC5); no longer U102.7 (SC1)
- net I2C1_{SDA}: now also U102.15 (SD5); no longer U102.6 (SD1)
- net I2C2_{SCL}: now also U102.14 (SC4); no longer U102.9 (SC2)
- net I2C2_{SDA}: now also U102.13 (SD4); no longer U102.8 (SD2)
- net I2C4_{SCL}: now also U102.9 (SC2); no longer U102.14 (SC4)
- net I2C4_{SDA}: now also U102.8 (SD2); no longer U102.13 (SD4)
- net I2C5_{SCL}: now also U102.7 (SC1); no longer U102.16 (SC5)
- net I2C5_{SDA}: now also U102.6 (SD1); no longer U102.15 (SD5)
- net I2C6_{SCL}: now also U102.5 (SC0); no longer U102.18 (SC6)
- net I2C6_{SDA}: now also U102.4 (SD0); no longer U102.17 (SD6)
- net MOD0_{GP0}: now also U2901.77 (P48); no longer U2901.3 (P0)
- net MOD0_{GP1}: now also U2901.78 (P49); no longer U2901.4 (P1)
- net MOD0_{GP2}: now also U2901.80 (P50); no longer U2901.6 (P2)
- net MOD0_{GP3}: now also U2901.81 (P51); no longer U2901.7 (P3)
- net MOD0_{GP4}: now also U2901.83 (P52); no longer U2901.9 (P4)
- net MOD0_{GP5}: now also U2901.84 (P53); no longer U2901.10 (P5)
- net MOD0_{GP6}: now also U2901.86 (P54); no longer U2901.12 (P6)
- net MOD0_{GP7}: now also U2901.87 (P55); no longer U2901.13 (P7)
- net MOD1_{GP0}: now also U2901.65 (P40); no longer U2901.15 (P8)
- net MOD1_{GP1}: now also U2901.66 (P41); no longer U2901.16 (P9)
- net MOD1_{GP2}: now also U2901.68 (P42); no longer U2901.18 (P10)
- net MOD1_{GP3}: now also U2901.69 (P43); no longer U2901.19 (P11)
- net MOD1_{GP4}: now also U2901.71 (P44); no longer U2901.21 (P12)
- net MOD1_{GP5}: now also U2901.72 (P45); no longer U2901.22 (P13)
- net MOD1_{GP6}: now also U2901.74 (P46); no longer U2901.24 (P14)
- net MOD1_{GP7}: now also U2901.75 (P47); no longer U2901.25 (P15)
- net MOD2_{GP0}: now also U2901.53 (P32); no longer U2901.27 (P16)
- net MOD2_{GP1}: now also U2901.54 (P33); no longer U2901.28 (P17)
- net MOD2_{GP2}: now also U2901.56 (P34); no longer U2901.30 (P18)
- net MOD2_{GP3}: now also U2901.57 (P35); no longer U2901.31 (P19)
- net MOD2_{GP4}: now also U2901.59 (P36); no longer U2901.33 (P20)
- net MOD2_{GP5}: now also U2901.60 (P37); no longer U2901.34 (P21)
- net MOD2_{GP6}: now also U2901.62 (P38); no longer U2901.36 (P22)
- net MOD2_{GP7}: now also U2901.63 (P39); no longer U2901.37 (P23)
- net MOD4_{GP0}: now also U2901.27 (P16); no longer U2901.53 (P32)
- net MOD4_{GP1}: now also U2901.28 (P17); no longer U2901.54 (P33)
- net MOD4_{GP2}: now also U2901.30 (P18); no longer U2901.56 (P34)
- net MOD4_{GP3}: now also U2901.31 (P19); no longer U2901.57 (P35)
- net MOD4_{GP4}: now also U2901.33 (P20); no longer U2901.59 (P36)
- net MOD4_{GP5}: now also U2901.34 (P21); no longer U2901.60 (P37)
- net MOD4_{GP6}: now also U2901.36 (P22); no longer U2901.62 (P38)
- net MOD4_{GP7}: now also U2901.37 (P23); no longer U2901.63 (P39)
- net MOD5_{GP0}: now also U2901.15 (P8); no longer U2901.65 (P40)
- net MOD5_{GP1}: now also U2901.16 (P9); no longer U2901.66 (P41)
- net MOD5_{GP2}: now also U2901.18 (P10); no longer U2901.68 (P42)
- net MOD5_{GP3}: now also U2901.19 (P11); no longer U2901.69 (P43)
- net MOD5_{GP4}: now also U2901.21 (P12); no longer U2901.71 (P44)
- net MOD5_{GP5}: now also U2901.22 (P13); no longer U2901.72 (P45)
- net MOD5_{GP6}: now also U2901.24 (P14); no longer U2901.74 (P46)
- net MOD5_{GP7}: now also U2901.25 (P15); no longer U2901.75 (P47)
- net MOD6_{GP0}: now also U2901.3 (P0); no longer U2901.77 (P48)
- net MOD6_{GP1}: now also U2901.4 (P1); no longer U2901.78 (P49)
- net MOD6_{GP2}: now also U2901.6 (P2); no longer U2901.80 (P50)
- net MOD6_{GP3}: now also U2901.7 (P3); no longer U2901.81 (P51)
- net MOD6_{GP4}: now also U2901.9 (P4); no longer U2901.83 (P52)
- net MOD6_{GP5}: now also U2901.10 (P5); no longer U2901.84 (P53)
- net MOD6_{GP6}: now also U2901.12 (P6); no longer U2901.86 (P54)
- net MOD6_{GP7}: now also U2901.13 (P7); no longer U2901.87 (P55)
- net P2_CLK: now also JP1.2 (B); no longer U3002.4 (Y)
- new net: JP1.1 (A), U3002.4 (Y)
