File: Hardware/Backplane.proto/mgmt_ctrl.kicad_sch (KiCad schematic)
At the start: 23 parts, among them J501 BM03B-SRSS-TB, Q501 S3134K, U502 CH32V003FxPx, U503 NL17SZS11DFT2G-Q

Commit message: Simplifies schematic and lays out PCB draft 1
Parts:
- removed C502, C503, C504: 100n, Capacitor_SMD:C_0603_1608Metric, symbol Device:C_Small
- removed J501: BM03B-SRSS-TB, Connector_JST:JST_SH_BM03B-SRSS-TB_1x03-1MP_P1.00mm_Vertical, symbol Connector_Generic:Conn_01x03
- removed Q501: S3134K, Package_TO_SOT_SMD:SOT-23, symbol Home Computer:S3134K
- removed R501, R509: 10K, Resistor_SMD:R_0603_1608Metric, symbol Device:R
- removed R502: 6K8 1%, Resistor_SMD:R_0603_1608Metric, symbol Device:R
- removed R503, R504, R505, R507: 1K8 1%, Resistor_SMD:R_0603_1608Metric, symbol Device:R
- removed R506: 560 1%, Resistor_SMD:R_0603_1608Metric, symbol Device:R
- removed R508, R510: 560, Resistor_SMD:R_0603_1608Metric, symbol Device:R
- removed TP2005, TP2013, TP2021, TP501, TP502: TestPoint_Small, TestPoint:TestPoint_Pad_D1.0mm, symbol Connector:TestPoint_Small
- removed U503: NL17SZS11DFT2G-Q, Package_TO_SOT_SMD:SOT-363_SC-70-6, symbol Home Computer:NL17SZS11DFT2G-Q
- added J6: Conn_01x03, Connector_PinHeader_2.54mm:PinHeader_1x03_P2.54mm_Vertical, symbol Connector_Generic:Conn_01x03
Connections:
- net MGMT_~{RST} is gone; now on net ~{RESET}: U502.4 (PD7)
- net DAP_SWIO: now also J6.1 (Pin_1)
- net GND: now also J6.3 (Pin_3)
- net OUT_{OC}: now also U502.15 (PC5)
- net ~{RESET}: now also J6.2 (Pin_2)
- net MEAS_+12V: no longer names the net of U502.1 (PD4)
- net MEAS_+3V3: no longer names the net of U502.3 (PD6)
- net MEAS_+5V: no longer names the net of U502.2 (PD5)
- no-connect marks 2 -> 5
Other:
- note removed: "12K"
- note removed: "3K3"
- note removed: "5K"
- note removed: "Debug Port"
- note removed: "~2.50 V"
- note removed: "~2.51 V"
