File: Hardware/Backplane.proto/module_slot.kicad_sch (KiCad schematic)
At the start: 29 parts, among them J402 10018784-10201TLF, Q401 S3134K, Q402 GSF3407, Q403 GSF3407, Q404 GSF3407, U401 NL17SZS11DFT2G-Q

Commit message: Simplifies schematic and lays out PCB draft 1
Parts:
- removed F401, F402, F403: SMD1206B050TF/15, Fuse:Fuse_1206_3216Metric, symbol Symbol Library:SMD1206B050TF/15
- removed Q401: S3134K, Package_TO_SOT_SMD:SOT-23, symbol Home Computer:S3134K
- removed Q402, Q403, Q404: GSF3407, Package_TO_SOT_SMD:SOT-23, symbol Home Computer:GSF3407
- removed R407, R411: 10K, Resistor_SMD:R_0603_1608Metric, symbol Device:R
- removed R408, R413: 560, Resistor_SMD:R_0603_1608Metric, symbol Device:R
- removed TP401, TP402, TP403: TestPoint_Small, TestPoint:TestPoint_Pad_D1.0mm, symbol Connector:TestPoint_Small
- removed U401: NL17SZS11DFT2G-Q, Package_TO_SOT_SMD:SOT-363_SC-70-6, symbol Home Computer:NL17SZS11DFT2G-Q
- added J15: Conn_02x03_Odd_Even, Connector_PinHeader_2.54mm:PinHeader_2x03_P2.54mm_Vertical, symbol Connector_Generic:Conn_02x03_Odd_Even
Connections:
- net MAIN_+12V: now also J15.1 (Pin_1)
- net MAIN_+3V3: now also J15.5 (Pin_5)
- net MAIN_+5V: now also J15.3 (Pin_3)
- net MOD_+12V: now also J15.2 (Pin_2)
- net MOD_+3V3: now also J15.6 (Pin_6)
- net MOD_+5V: now also J15.4 (Pin_4)
- no-connect marks 9 -> 11
Other:
- sheet Management Controller ports: added none; removed REF_+12V, REF_+3V3, REF_+5V
- moved on the sheet: D401, R412, TP407, TP408
