File: Hardware/Backplane.proto/power.kicad_sch (KiCad schematic)
At the start: 57 parts, among them J2902 Conn_02x08_Counter_Clockwise, U2901 P2X8C4M64P, U2902 AP3445LW6-7

Commit message: Simplifies schematic and lays out PCB draft 1
Parts:
- removed C2936, C2937: 22u, Capacitor_SMD:C_0603_1608Metric, symbol Device:C
- removed F2901, F2902, F2903: 0ZCF0400FF2A, Home Computer:FUSER_0ZCF0400FF2A, symbol Symbol Library:SMD1206B050TF/15
- removed J2902: Conn_02x08_Counter_Clockwise, Connector_PinHeader_2.54mm:PinHeader_2x08_P2.54mm_Vertical_SMD, symbol Connector_Generic:Conn_02x08_Odd_Even
- removed TP2901: +12V, TestPoint:TestPoint_Pad_D2.0mm, symbol Connector:TestPoint
- removed TP2902: +5V, TestPoint:TestPoint_Pad_D2.0mm, symbol Connector:TestPoint
- removed TP2903: +3V3, TestPoint:TestPoint_Pad_D2.0mm, symbol Connector:TestPoint
- removed TP2904, TP2905: +1V8, TestPoint:TestPoint_Pad_D2.0mm, symbol Connector:TestPoint
- added C2938, C2939: 22u, Capacitor_SMD:CP_Elec_4x5.4, symbol Device:C_Polarized
- added J14: Conn_01x06, Connector_PinHeader_2.54mm:PinHeader_1x06_P2.54mm_Vertical, symbol Connector_Generic:Conn_01x06
- C2901: footprint Capacitor_SMD:C_1206_3216Metric -> Capacitor_SMD:CP_Elec_6.3x9.9; symbol Device:C -> Device:C_Polarized; Digikey Part No 490-13970-1-ND -> 732-8492-1-ND
- TP2906: footprint Jumper:SolderJumper-2_P1.3mm_Open_Pad1.0x1.5mm -> Connector_PinHeader_2.54mm:PinHeader_1x02_P2.54mm_Vertical
Connections:
- net +5V: now also C2901.1; no longer C2901.2
- net GND: now also C2901.2, C2938.2, C2939.2; no longer C2901.1
- net MAIN_+12V: now also J14.1 (Pin_1)
- net MAIN_+3V3: now also J14.3 (Pin_3)
- net MAIN_+5V: now also J14.2 (Pin_2)
- net MAIN_GND: now also J14.5 (Pin_5), J14.6 (Pin_6)
- net POWER_OK: now also J14.4 (Pin_4)
- net at C2935.2, L2901.2, R2901.2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: now also C2938.1, C2939.1
- no-connect marks 1 -> 0
Other:
- note removed: "Solder when power OK"
