File: Hardware/Backplane.proto/usb_socket.kicad_sch (KiCad schematic)
At the start: 7 parts, among them J2102 Molex 105057

Commit message: Simplifies schematic and lays out PCB draft 1
Parts:
- removed F2101: SMD1206B050TF/15, Fuse:Fuse_1206_3216Metric, symbol Symbol Library:SMD1206B050TF/15
- removed J2102: Molex 105057, Connector_USB:USB_A_Molex_105057_Vertical, symbol Connector:USB_A
- removed R2102, R2103: 0, Resistor_SMD:R_0603_1608Metric, symbol Device:R_Small
- removed TP2103, TP2104, TP2105: TestPoint_Small, TestPoint:TestPoint_Pad_D1.0mm, symbol Connector:TestPoint_Small
- added J2: (no value), Connector_PinHeader_2.54mm:PinHeader_1x04_P2.54mm_Vertical, symbol Connector_Generic:Conn_01x04
Connections:
- net D+: now also J2.2 (Pin_2)
- net D-: now also J2.3 (Pin_3)
- net GND: now also J2.4 (Pin_4)
- new net +5V: J2.1 (Pin_1)
Other:
- note removed: "0 Ohm"
